File: HARDWARE/pnp32_controller/pnp32_mainboard/PSU.kicad_sch (KiCad schematic)
At the start: 0 parts

Commit message: update
Parts:
- added C1, C19, C26, C30, C36, C37: 100nF, fab_C:C_0402, symbol fab_C:C_100nF_0402
- added C13: 100nF, fab_C:C_0603, symbol fab_C:C_100nF_0603_16V
- added C20, C21, C23: 10uF, fab_C:C_1210, symbol fab_C:C_10uF_1210_50V
- added C22, C25: 1uF, fab_C:C_0603, symbol fab_C:C_1uF_0603_50V
- added C24, C29: 1uF, fab_C:C_0603, symbol fab_C:C_1uF_0603
- added C27: 10pF, fab_C:C_0603, symbol fab_C:C_10pF_0603
- added C28: 100uF, fab_C:C_1206, symbol fab_C:C_100uF_1206
- added C31: 100nF, fab_C:C_0805, symbol fab_C:C_100nF_0805
- added C32: 10uF, fab_C:C_1206, symbol fab_C:C_10uF_1206
- added C33, SCAP1, SCAP2: C_Polarized, symbol Device:C_Polarized
- added C34: 2.2uF, fab_C:C_0603, symbol fab_C:C_2.2uF_0603
- added C35: 1nF, fab_C:C_0402, symbol fab_C:C_1nF_0402
- added C38: 10uF, fab_C:C_0603, symbol fab_C:C_10uF_0603_10V
- added C39, C40: 100uF, fab_C:C_1210, symbol fab_C:C_100uF_1210
- added C7: 22uF/63V, fab_C_Pol:CP_Elec_6.3x7.7, symbol fab_C_Pol:C_Pol_22uF_D6.3xL7.7mm
- added D1, D2: KT-0603Y, fab_D:LED_0603_1608Metric, symbol fab_D:KT-0603Y
- added D3: KT-0603R, fab_D:LED_0603_1608Metric, symbol fab_D:KT-0603R
- added D4: BAS40-05-7-F, fab_D:SOT23-3, symbol fab_D:BAS40-05-7-F
- added FB1: MPZ1608S300ATAH0, fab_R:R_0603, symbol fab_L:MPZ1608S300ATAH0
- added JP1, JP2, JP3: SolderJumper_2_Open, Jumper:SolderJumper-2_P1.3mm_Open_TrianglePad1.0x1.5mm, symbol Jumper:SolderJumper_2_Open
- added JP4, JP5: SolderJumper_3_Open, Jumper:SolderJumper-3_P2.0mm_Open_TrianglePad1.0x1.5mm_NumberLabels, symbol Jumper:SolderJumper_3_Open
- added L1, L2: L, symbol Device:L
- added L3: 2.2uH, fab_L:L_Coilcraft_XAL5030-XXX, symbol fab_L:L_2.2uH_SMD,5.2x5.4mm
- added R1, R6: 100kΩ, fab_R:R_0603, symbol fab_R:R_100kΩ_0603
- added R10, R11, R9: 1.5kΩ, fab_R:R_0402, symbol fab_R:R_1.5kΩ_0402
- added R12: 113kΩ, fab_R:R_0402, symbol fab_R:R_113kΩ_0402
- added R13: 38.3kΩ, fab_R:R_0402, symbol fab_R:R_38.3kΩ_0402
- added R14: 6.2kΩ, fab_R:R_0603, symbol fab_R:R_6.2kΩ_0603
- added R15: 1kΩ, fab_R:R_0603, symbol fab_R:R_1kΩ_0603
- added R16, R4: 0Ω, fab_R:R_0603, symbol fab_R:R_0Ω_0603
- added R17: 324kΩ, fab_R:R_0402, symbol fab_R:R_324kΩ_0402
- added R18: 1.5MΩ, fab_R:R_0402, symbol fab_R:R_ 1.5MΩ_0402
- added R19: 1.05MΩ, fab_R:R_0402, symbol fab_R:R_1.05MΩ_0402
- added R2: 17.8kΩ, fab_R:R_0603, symbol fab_R:R_17.8kΩ_0603
- added R20: 200kΩ, fab_R:R_0402, symbol fab_R:R_200kΩ_0402
- added R21: 0Ω, fab_R:R_0402, symbol fab_R:R_0Ω_0402
- added R22, R7, R8: 1MΩ, fab_R:R_0402, symbol fab_R:R_1MΩ_0402
- added R3: 1MΩ, fab_R:R_0603, symbol fab_R:R_1MΩ_0603
- added R5: 243kΩ, fab_R:R_0603, symbol fab_R:R_243kΩ_0603
- added U2: LT8637, fab_U:LQFN-20-1EP_3x4mm_P0.5mm_EP1.65x2.65mm, symbol fab_U:LT8637JV#WPBF
- added U8: LTC4041, fab_U:QFN-24-1EP_4x5mm_P0.5mm_EP2.65x3.65mm, symbol fab_U:LTC4041
Connections:
- new net: D4.3 (K), JP4.3 (B), JP5.3 (B)
- new net: R17.1, R18.1, U8.12 (CAPFB)
- new net: C26.1, L2.1, U2.10 (SW), U2.8 (SW), U2.9 (SW)
- new net: C20.1, C22.1, C25.1, C7.1, L1.2, R1.1, U2.11 (VIN), U2.6 (VIN)
- new net: JP1.2 (B), JP2.2 (B), JP3.2 (B), U2.15 (SYNC/MODE)
- new net: R2.1, U2.17 (RT)
- new net: R4.1, U2.2 (BIAS)
- new net: C27.2, R3.2, R5.1, U2.20 (FB)
- new net: C24.1, JP3.1 (A), U2.3 (INTVCC)
- new net: C26.2, U2.7 (BST)
- new net: R19.2, R20.1, R21.1, U8.18 (BSTFB)
- new net: R21.2, U8.10 (RSTFB)
- new net: R14.2, U8.16 (OVSNS)
- new net: C35.1, U8.17 (CPF)
- new net: R12.2, R13.1, U8.19 (PFI)
- new net: R15.1, R22.2, U8.2 (PROG)
- new net: R16.2, U8.20 (CAPSEL)
- new net: L3.1, U8.21 (SW), U8.22 (SW)
- new net: R8.1, U8.3 (IMON)
- new net: C30.1, R10.1, R11.1, R7.1, R9.1
- new net: C23.1, FB1.2, L1.1
- new net: D2.2 (A), R10.2
- new net: D3.2 (A), R11.2
- new net: D1.2 (A), R9.2
- new net BAL: SCAP1.2, SCAP2.1, U8.9 (BAL)
- new net CAPGD: D1.1 (K), U8.13 (CAPGD)
- new net CLKOUT: U2.16 (CLKOUT)
- new net DCIN: C27.1, C28.1, C29.1, C31.1, C32.1, C33.1, L2.2, R12.1, R14.1, R3.1, R4.2, R6.1
- new net EN: R1.2, U2.14 (EM/UV)
- new net GND: C1.2, C13.2, C19.2, C20.2, C21.2, C22.2, C23.2, C24.2, C25.2, C28.2, C29.2, C30.2, C31.2, C32.2, C33.2, C34.2, C35.2, C36.2, C37.2, C38.2, C39.2, C40.2, C7.2, JP2.1 (A), JP4.1 (A), JP5.1 (A), R13.2, R15.2, R17.2, R2.2, R20.2, R5.2, SCAP2.2, U2.12 (NC), U2.13 (GND), U2.21 (GND), U2.4 (GND), U2.5 (NC), U8.25 (GND)
- new net IMON: R8.2
- new net PG: R6.2, U2.1 (PG)
- new net PROG: R22.1
- new net SCAP: C37.1, C38.1, D4.1 (A), L3.2, R18.2, SCAP1.1, U8.23 (SCAP)
- new net SYNC: JP1.1 (A)
- new net SYSGD: D3.1 (K), U8.11 (SYSGD)
- new net TR/SS: C13.1, U2.18 (TR/SS)
- new net VEMI: C1.1, C19.1, C21.1, FB1.1
- new net VSYS: C36.1, C39.1, C40.1, D4.2 (A), R16.1, R19.1, U8.1 (VSYS), U8.24 (VSYS)
- new net ~{BSTEN}: JP5.2 (C), U8.5 (~{BSTEN})
- new net ~{CAPFLT}: R7.2, U8.8 (~{CAPFLT})
- new net ~{CHGEN}: JP4.2 (C), U8.4 (~{CHGEN})
- new net ~{PFO}: D2.1 (K), U8.14 (~{PFO})
Other:
- note added: "VSYS alebo EXTVDD ktore sa urcovalo switchom"
- company: (none) -> telelmetry.digital s.r.o.
- title: (none) -> pnp32 Motion Controller

Commit message: update
Parts:
- removed C1, C19, C26, C30, C36, C37: 100nF, fab_C:C_0402, symbol fab_C:C_100nF_0402
- removed C13: 100nF, fab_C:C_0603, symbol fab_C:C_100nF_0603_16V
- removed C20, C21, C23: 10uF, fab_C:C_1210, symbol fab_C:C_10uF_1210_50V
- removed C22, C25: 1uF, fab_C:C_0603, symbol fab_C:C_1uF_0603_50V
- removed C24, C29: 1uF, fab_C:C_0603, symbol fab_C:C_1uF_0603
- removed C27: 10pF, fab_C:C_0603, symbol fab_C:C_10pF_0603
- removed C28: 100uF, fab_C:C_1206, symbol fab_C:C_100uF_1206
- removed C31: 100nF, fab_C:C_0805, symbol fab_C:C_100nF_0805
- removed C32: 10uF, fab_C:C_1206, symbol fab_C:C_10uF_1206
- removed C33, SCAP1, SCAP2: C_Polarized, symbol Device:C_Polarized
- removed C34: 2.2uF, fab_C:C_0603, symbol fab_C:C_2.2uF_0603
- removed C35: 1nF, fab_C:C_0402, symbol fab_C:C_1nF_0402
- removed C38: 10uF, fab_C:C_0603, symbol fab_C:C_10uF_0603_10V
- removed C39, C40: 100uF, fab_C:C_1210, symbol fab_C:C_100uF_1210
- removed C7: 22uF/63V, fab_C_Pol:CP_Elec_6.3x7.7, symbol fab_C_Pol:C_Pol_22uF_D6.3xL7.7mm
- removed D1, D2: KT-0603Y, fab_D:LED_0603_1608Metric, symbol fab_D:KT-0603Y
- removed D3: KT-0603R, fab_D:LED_0603_1608Metric, symbol fab_D:KT-0603R
- removed D4: BAS40-05-7-F, fab_D:SOT23-3, symbol fab_D:BAS40-05-7-F
- removed FB1: MPZ1608S300ATAH0, fab_R:R_0603, symbol fab_L:MPZ1608S300ATAH0
- removed JP1, JP2, JP3: SolderJumper_2_Open, Jumper:SolderJumper-2_P1.3mm_Open_TrianglePad1.0x1.5mm, symbol Jumper:SolderJumper_2_Open
- removed JP4, JP5: SolderJumper_3_Open, Jumper:SolderJumper-3_P2.0mm_Open_TrianglePad1.0x1.5mm_NumberLabels, symbol Jumper:SolderJumper_3_Open
- removed L1, L2: L, symbol Device:L
- removed L3: 2.2uH, fab_L:L_Coilcraft_XAL5030-XXX, symbol fab_L:L_2.2uH_SMD,5.2x5.4mm
- removed R1, R6: 100kΩ, fab_R:R_0603, symbol fab_R:R_100kΩ_0603
- removed R10, R11, R9: 1.5kΩ, fab_R:R_0402, symbol fab_R:R_1.5kΩ_0402
- removed R12: 113kΩ, fab_R:R_0402, symbol fab_R:R_113kΩ_0402
- removed R13: 38.3kΩ, fab_R:R_0402, symbol fab_R:R_38.3kΩ_0402
- removed R14: 6.2kΩ, fab_R:R_0603, symbol fab_R:R_6.2kΩ_0603
- removed R15: 1kΩ, fab_R:R_0603, symbol fab_R:R_1kΩ_0603
- removed R16, R4: 0Ω, fab_R:R_0603, symbol fab_R:R_0Ω_0603
- removed R17: 324kΩ, fab_R:R_0402, symbol fab_R:R_324kΩ_0402
- removed R18: 1.5MΩ, fab_R:R_0402, symbol fab_R:R_ 1.5MΩ_0402
- removed R19: 1.05MΩ, fab_R:R_0402, symbol fab_R:R_1.05MΩ_0402
- removed R2: 17.8kΩ, fab_R:R_0603, symbol fab_R:R_17.8kΩ_0603
- removed R20: 200kΩ, fab_R:R_0402, symbol fab_R:R_200kΩ_0402
- removed R21: 0Ω, fab_R:R_0402, symbol fab_R:R_0Ω_0402
- removed R22, R7, R8: 1MΩ, fab_R:R_0402, symbol fab_R:R_1MΩ_0402
- removed R3: 1MΩ, fab_R:R_0603, symbol fab_R:R_1MΩ_0603
- removed R5: 243kΩ, fab_R:R_0603, symbol fab_R:R_243kΩ_0603
- removed U2: LT8637, fab_U:LQFN-20-1EP_3x4mm_P0.5mm_EP1.65x2.65mm, symbol fab_U:LT8637JV#WPBF
- removed U8: LTC4041, fab_U:QFN-24-1EP_4x5mm_P0.5mm_EP2.65x3.65mm, symbol fab_U:LTC4041
Other:
- note removed: "VSYS alebo EXTVDD ktore sa urcovalo switchom"

Commit message: update
Parts:
- added C1, C8: 100n, Capacitor_SMD:C_0805_2012Metric, symbol Device:C_Small
- added C10, C12, C13, C15, C17, C18, C2, C3, C4, C5, C7, C9: 10u, Capacitor_SMD:C_0805_2012Metric, symbol Device:C_Small
- added C11, C6: 100u, Capacitor_SMD:CP_Elec_6.3x7.7, symbol Device:C_Polarized_Small
- added C14: 47p, Capacitor_SMD:C_0805_2012Metric, symbol Device:C_Small
- added C16: 4.7n, Capacitor_SMD:C_0805_2012Metric, symbol Device:C_Small
- added D1, D2: BZT52C16, Diode_SMD:D_SOD-123, symbol Diode:BZT52Bxx
- added D3: SMF28A, Diode_SMD:D_SMF, symbol Diode:SMF28A
- added D4: B560C, Diode_SMD:D_SMC, symbol Device:D_Schottky
- added D6, D7, D8: Green, LED_SMD:LED_0805_2012Metric, symbol Device:LED_Small
- added F1: Fuse, Fuse:Fuseholder_Littelfuse_Nano2_154x, symbol Device:Fuse
- added J1: COMBO_POWER_JACK, index:BarrelJack_Horizontal, symbol Connector:Conn_01x04_Male
- added L1: 2.2u, Inductor_SMD:L_Sunlord_MWSA0402S, symbol Device:L
- added L2: 8.2uH, Inductor_SMD:L_Sunlord_MWSA0603S, symbol Device:L
- added R1, R12, R2, R8: 4.7k, Resistor_SMD:R_0805_2012Metric, symbol Device:R_Small
- added R10, R11, R3, R4, R5: 10k, Resistor_SMD:R_0805_2012Metric, symbol Device:R_Small
- added R13: 1k, Resistor_SMD:R_0805_2012Metric, symbol Device:R_Small
- added R6: 53.6k, Resistor_SMD:R_0805_2012Metric, symbol Device:R_Small
- added R7: 16.9k, Resistor_SMD:R_0805_2012Metric, symbol Device:R_Small
- added R9: 243k, Resistor_SMD:R_0805_2012Metric, symbol Device:R_Small
- added TP1, TP2, TP3, TP4, TP5: TestPoint, TestPoint:TestPoint_Pad_D2.0mm, symbol Connector:TestPoint
- added U1, U2: FDS4435BZ, Package_SO:SO-8_3.9x4.9mm_P1.27mm, symbol index:FDS4435BZ
- added U3: TPS54560BDDA, Package_SO:Texas_R-PDSO-G8_EP2.95x4.9mm_Mask2.4x3.1mm_ThermalVias, symbol Regulator_Switching:TPS54560BDDA
- added U4: AP1117-33, Package_TO_SOT_SMD:SOT-223-3_TabPin2, symbol Regulator_Linear:AP1117-33
Connections:
- new net: D8.2 (A), R13.2
- new net: C1.1, D2.2 (A), R2.2, R4.1, U2.4 (G)
- new net: R5.2, R8.1, U3.3 (EN)
- new net: D6.2 (A), R11.2
- new net: D7.2 (A), R12.2
- new net: C8.1, D4.1 (K), L2.1, U3.8 (SW)
- new net: C1.2, D1.1 (K), D2.1 (K), R1.1, R2.1, U1.1 (S), U1.2 (S), U1.3 (S), U2.1 (S), U2.2 (S), U2.3 (S)
- new net: D1.2 (A), R1.2, R3.1, U1.4 (G)
- new net: C8.2, U3.1 (BOOT)
- new net: R9.1, U3.4 (RT/CLK)
- new net: R10.1, R6.2, U3.5 (FB)
- new net: C14.2, R7.1, U3.6 (COMP)
- new net: C2.2, C3.2, L1.1, U2.5 (D), U2.6 (D), U2.7 (D), U2.8 (D)
- new net: C16.2, R7.2
- new net +3.3V: C18.1, R13.1, TP5.1, U4.2 (VO)
- new net +5V: C10.2, C11.1, C13.2, C15.2, C17.1, L2.2, R12.1, R6.1, TP4.1, U4.3 (VI)
- new net GND: C10.1, C11.2, C12.1, C13.1, C14.1, C15.1, C16.1, C17.2, C18.2, C2.1, C3.1, C4.1, C5.1, C6.2, C7.1, C9.1, D3.2 (A2), D4.2 (A), D6.1 (K), D7.1 (K), D8.1 (K), J1.2 (Pin_2), J1.3 (Pin_3), R10.2, R3.2, R4.2, R8.2, R9.2, TP3.1, U3.7 (GND), U3.9 (GND), U4.1 (GND)
- new net POWER_SUPPLY: F1.1, J1.1 (Pin_1), J1.4 (Pin_4)
- new net VDC: C12.2, C4.2, C5.2, C6.1, C9.2, L1.2, R11.1, R5.1, TP2.1, U3.2 (VIN)
- new net VIN: C7.2, D3.1 (A1), F1.2, TP1.1, U1.5 (D), U1.6 (D), U1.7 (D), U1.8 (D)
Other:
- note added: "3V3 linear regulator"
- note added: "PSU active LED"
- note added: "VCC_P"
