File: HARDWARE/pnp32_controller/pnp32_mainboard/pnp32_mainboard.kicad_sch (KiCad schematic)
At the start: 0 parts

Commit message: update
Other:
- removed sheet Y_L-driver
- removed sheet Y_R-driver
- added sheet A-driver (driver_TMC5130.kicad_sch)
- added sheet B-driver (driver_TMC5130.kicad_sch)
- added sheet C-driver (driver_TMC5130.kicad_sch)
- added sheet Y-driver (driver_TMC5130.kicad_sch)
- added sheet Z-driver (driver_TMC5130.kicad_sch)
- sheet CPU ports: added I2C_SCL, I2C_SDA, SPI_CLK, SPI_CS_A, SPI_CS_B, SPI_CS_C, SPI_CS_X, SPI_CS_Y, SPI_CS_Z, SPI_MISO, SPI_MOSI; removed none
- sheet X-driver ports: added SPI_CLK, SPI_CS, SPI_MISO, SPI_MOSI; removed none

Commit message: update
Other:
- removed sheet X-driver
- company: (none) -> telelmetry.digital s.r.o.
- title: (none) -> pnp32 Motion Controller
Changed lines of the file:
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@@
 	(generator_version "9.0")
 	(paper "A4")
+	(title_block
+		(title "pnp32 Motion Controller")
+		(date "2025-08-01")
+		(rev "V0.1")
+		(company "telelmetry.digital s.r.o.")
+	)
 	(junction
 		(at 236.22 101.6)
@@
 				)
 			)
-		)
-	)
-	(sheet
-		(at 245.11 20.32)
-		(size 33.02 12.7)
-		(exclude_from_sim no)
-		(in_bom yes)
-		(on_board yes)
-		(dnp no)
-		(fields_autoplaced yes)
-		(stroke
-			(width 0.1524)
-			(type solid)
-		)
-		(fill
-			(color 0 0 0 0.0000)
-		)
-		(property "Sheetname" "X-driver"
-			(at 245.11 19.6084 0)
-			(effects
-				(font
-					(size 1.27 1.27)
-				)
-				(justify left bottom)
-			)
-		)
-		(property "Sheetfile" "driver_TMC5130.kicad_sch"
-			(at 245.11 33.6046 0)
-			(effects
-				(font
-					(size 1.27 1.27)
-				)
-				(justify left top)
-			)
-		)
-		(pin "SPI_CLK" input
-			(at 245.11 27.94 180)
-			(effects
-				(font
-					(size 1.27 1.27)
-				)
-				(justify left)
-			)
-		)
-		(pin "SPI_CS" input
-			(at 245.11 30.48 180)
-			(effects
-				(font
-					(size 1.27 1.27)
-				)
-				(justify left)
-			)
-		)
-		(pin "SPI_MISO" input
-			(at 245.11 22.86 180)
-			(effects
-				(font
-					(size 1.27 1.27)
-				)
-				(justify left)
-			)
-		)
-		(pin "SPI_MOSI" input
-			(at 245.11 25.4 180)
-			(effects
-				(font
-					(size 1.27 1.27)
-				)
-				(justify left)
-			)
-		)
-		(instances
-			(project "pnp32_mainboard"
-				(path "/a02e5dd1-80da-4253-b87a-c8707aa3e0b0"
-					(page "4")
-				)
-			)

Commit message: update
Other:
- added sheet X-driver (driver_TMC5130.kicad_sch)
Changed lines of the file:
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@@
 			(project "pnp32_mainboard"
 				(path "/a02e5dd1-80da-4253-b87a-c8707aa3e0b0"
-					(page "8")
+					(page "6")
+				)
+			)
+		)
+	)
+	(sheet
+		(at 245.11 20.32)
+		(size 33.02 12.7)
+		(exclude_from_sim no)
+		(in_bom yes)
+		(on_board yes)
+		(dnp no)
+		(fields_autoplaced yes)
+		(stroke
+			(width 0.1524)
+			(type solid)
+		)
+		(fill
+			(color 0 0 0 0.0000)
+		)
+		(property "Sheetname" "X-driver"
+			(at 245.11 19.6084 0)
+			(effects
+				(font
+					(size 1.27 1.27)
+				)
+				(justify left bottom)
+			)
+		)
+		(property "Sheetfile" "driver_TMC5130.kicad_sch"
+			(at 245.11 33.6046 0)
+			(effects
+				(font
+					(size 1.27 1.27)
+				)
+				(justify left top)
+			)
+		)
+		(pin "SPI_CLK" input
+			(at 245.11 27.94 180)
+			(effects
+				(font
+					(size 1.27 1.27)
+				)
+				(justify left)
+			)
+		)
+		(pin "SPI_CS" input
+			(at 245.11 30.48 180)
+			(effects
+				(font
+					(size 1.27 1.27)
+				)
+				(justify left)
+			)
+		)
+		(pin "SPI_MISO" input
+			(at 245.11 22.86 180)
+			(effects
+				(font
+					(size 1.27 1.27)
+				)
+				(justify left)
+			)
+		)
+		(pin "SPI_MOSI" input
+			(at 245.11 25.4 180)
+			(effects
+				(font
+					(size 1.27 1.27)
+				)
+				(justify left)
+			)
+		)
+		(instances
+			(project "pnp32_mainboard"
+				(path "/a02e5dd1-80da-4253-b87a-c8707aa3e0b0"
+					(page "4")
 				)
 			)
@@
 			(project "pnp32_mainboard"
 				(path "/a02e5dd1-80da-4253-b87a-c8707aa3e0b0"
-					(page "7")
-				)
-			)
+					(page "5")
+				)
+			)

Commit message: update
Parts:
- added FID1, FID2, FID3, FID4: Fiducial, Fiducial:Fiducial_1mm_Mask2mm, symbol Mechanical:Fiducial
- added H1, H2, H3, H4: MountingHole_Pad, MountingHole:MountingHole_3.2mm_M3_DIN965_Pad, symbol Mechanical:MountingHole_Pad
Connections:
- new net GND: H1.1, H2.1, H3.1, H4.1
Other:
- added sheet AIR1 (mosfet.kicad_sch)
- added sheet AIR2 (mosfet.kicad_sch)
- added sheet AIR_PUMP (mosfet.kicad_sch)
- added sheet E-STOP (digital_input.kicad_sch)
- added sheet ENABLE (digital_input.kicad_sch)
- added sheet LIGHT_BOTTOM (wled.kicad_sch)
- added sheet LIGHT_TOP (wled.kicad_sch)
- added sheet VAC1 (mosfet.kicad_sch)
- added sheet VAC2 (mosfet.kicad_sch)
- added sheet VAC_PUMP (mosfet.kicad_sch)
- added sheet X_STOP (digital_input.kicad_sch)
- added sheet Y_STOP (digital_input.kicad_sch)
- added sheet Z_STOP (digital_input.kicad_sch)
- sheet CPU ports: added AIR1, AIR2, AIR_PUMP, E-STOP, ENABLE, LIGHT_BOTTOM, LIGHT_TOP, VAC1, VAC2, VAC_PUMP, X_STOP, Y_STOP, Z_STOP; removed none
- note added: "Pridať -USB Hub FE1.11s + CH340X - 2x usb vystup a treti na CH340 - RS485 - odkreslit z displejov - vakuovy senzor najst s I2C SMD na podtlak vakuum a dobre bybolo aj na tlak - wled odkresliť z SKR + pridať ESD ochranu - digitalne tranzistorove vystupy mosfet zmeniť tranzistory na pumpach s vacsim vykonom - dorobit drivery - schema tu --- https://www.mikroe.com/silent-step-click - nie sú dorobené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"
- note added: "pnp32 - openPNP Motion Controller"
