File: HARDWARE/pnp32_controller/pnp32_mainboard/digital_input.kicad_sch (KiCad schematic)
At the start: 4 parts, among them J17 TOP_LIGHT

Commit message: update_PSU
Parts:
- removed J17: TOP_LIGHT, Connector_JST:JST_PH_B3B-PH-SM4-TB_1x03-1MP_P2.00mm_Vertical, symbol Connector_Generic_MountingPin:Conn_01x03_MountingPin
- added J17: Conn_01x03_Pin, fab_CON:WE_620303124022, symbol fab_CON:WE_620303124022
- renumbered D17 to D19, R40 to R44
Connections:
- net +5V: now also J17.1 (Pin_1)
- net GND: now also J17.3 (Pin_3)
- net at D19.2 (A2), R44.2, R45.2: now also J17.2 (Pin_2)
