File: HARDWARE/pnp32_controller/pnp32_mainboard/driver_TMC5130.kicad_sch (KiCad schematic)
At the start: 1 part, among them U2 TMC5130A-TA

Commit message: update
Changed lines of the file:
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@@
 		)
 	)
-	(global_label "SPI_CLK"
+	(hierarchical_label "SPI_MISO"
+		(shape input)
+		(at 45.72 74.93 180)
+		(effects
+			(font
+				(size 1.27 1.27)
+			)
+			(justify right)
+		)
+	)
+	(hierarchical_label "SPI_CLK"
 		(shape input)
 		(at 45.72 69.85 180)
-		(fields_autoplaced yes)
-		(effects
-			(font
-				(size 1.27 1.27)
-			)
-			(justify right)
-		)
-		(property "Intersheetrefs" "${INTERSHEET_REFS}"
-			(at 35.1148 69.85 0)
-			(effects
-				(font
-					(size 1.27 1.27)
-				)
-				(justify right)
-				(hide yes)
-			)
-		)
-	)
-	(global_label "SPI_CS"
+		(effects
+			(font
+				(size 1.27 1.27)
+			)
+			(justify right)
+		)
+	)
+	(hierarchical_label "SPI_MOSI"
+		(shape input)
+		(at 45.72 72.39 180)
+		(effects
+			(font
+				(size 1.27 1.27)
+			)
+			(justify right)
+		)
+	)
+	(hierarchical_label "SPI_CS"
 		(shape input)
 		(at 45.72 67.31 180)
-		(fields_autoplaced yes)
-		(effects
-			(font
-				(size 1.27 1.27)
-			)
-			(justify right)
-		)
-		(property "Intersheetrefs" "${INTERSHEET_REFS}"
-			(at 36.2034 67.31 0)
-			(effects
-				(font
-					(size 1.27 1.27)
-				)
-				(justify right)
-				(hide yes)
-			)
-		)
-	)
-	(global_label "SPI_MOSI"
-		(shape input)
-		(at 45.72 72.39 180)
-		(fields_autoplaced yes)
-		(effects
-			(font
-				(size 1.27 1.27)
-			)
-			(justify right)
-		)
-		(property "Intersheetrefs" "${INTERSHEET_REFS}"
-			(at 34.0867 72.39 0)
-			(effects
-				(font
-					(size 1.27 1.27)
-				)
-				(justify right)
-				(hide yes)
-			)
-		)
-	)
-	(global_label "SPI_MISO"
-		(shape input)
-		(at 45.72 74.93 180)
-		(fields_autoplaced yes)
-		(effects
-			(font
-				(size 1.27 1.27)
-			)
-			(justify right)
-		)
-		(property "Intersheetrefs" "${INTERSHEET_REFS}"
-			(at 34.0867 74.93 0)
-			(effects
-				(font
-					(size 1.27 1.27)
-				)
-				(justify right)
-				(hide yes)
-			)
+		(effects
+			(font
+				(size 1.27 1.27)
+			)
+			(justify right)
 		)
 	)
@@
 		(instances
 			(project "pnp32_mainboard"
-				(path "/a02e5dd1-80da-4253-b87a-c8707aa3e0b0/587aa0d5-267c-4288-a48c-61def213ea86"
-					(reference "U4")
-					(unit 1)
-				)
-				(path "/a02e5dd1-80da-4253-b87a-c8707aa3e0b0/9805ec31-9a99-4e4b-a625-8fd11a9a458a"
-					(reference "U3")
+				(path "/a02e5dd1-80da-4253-b87a-c8707aa3e0b0/36c8ee69-d46e-4392-9648-7ffe454aa773"
+					(reference "U6")
+					(unit 1)
+				)
+				(path "/a02e5dd1-80da-4253-b87a-c8707aa3e0b0/4927e2a7-a4c2-4e52-af67-49600773c73d"
+					(reference "U5")
+					(unit 1)
+				)
+				(path "/a02e5dd1-80da-4253-b87a-c8707aa3e0b0/831bc4de-0744-4eeb-b882-33b45fc786ec"
+					(reference "U7")
 					(unit 1)
 				)
@@
 					(unit 1)
 				)
+				(path "/a02e5dd1-80da-4253-b87a-c8707aa3e0b0/a54d937e-12a5-4dff-8c5d-763d1b46ce81"
+					(reference "U3")
+					(unit 1)
+				)
+				(path "/a02e5dd1-80da-4253-b87a-c8707aa3e0b0/bc306ebc-9231-4e41-974d-f78f75c244a9"
+					(reference "U4")
+					(unit 1)
+				)

Commit message: update
Parts:
- removed U2: TMC5130A-TA, Package_QFP:TQFP-48-1EP_7x7mm_P0.5mm_EP5x5mm_ThermalVias, symbol Driver_Motor:TMC5130A-TA
- added C1: 22nF/0805, fab_C:C_0805, symbol fab_C:C_100nF_0805
- added C13: 470nF, fab_C:C_0603, symbol fab_C:C_75pF_0603
- added C7: 4.7uF, fab_C:C_0603, symbol fab_C:C_4.7uF_0603
- added U2: TMC5130A-TA, fab_U:TQFP-48-1EP_7x7mm_P0.5mm_EP5x5mm_ThermalVias, symbol fab_U:TMC5130A-TA-T
Connections:
- net SPI_CLK: now also U2.4 (SCK_CFG2)
- net SPI_CS: now also U2.3 (~{CS}_CFG3)
- net SPI_MISO: now also U2.7 (SDO_NAO_CFG0)
- net SPI_MOSI: now also U2.5 (SDI_NAI_CFG1)
- new net: U2.13 (GNDP), U2.48 (GNDP)
- new net: C7.1, U2.33 (5VOUT)
- new net: C13.1, U2.34 (VCC)
- new net CPI: C1.2, U2.37 (CPI)
- new net CPO: C1.1, U2.35 (CP0)
- new net GND: C13.2, C7.2
- no-connect marks 0 -> 3

Commit message: update
Parts:
- renumbered C13 to C14, C1 to C2, C7 to C8, U2 to U3
Other:
- company: (none) -> telelmetry.digital s.r.o.
- title: (none) -> pnp32 Motion Controller
Changed lines of the file:
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@@
 	(generator_version "9.0")
 	(paper "A4")
+	(title_block
+		(title "pnp32 Motion Controller")
+		(date "2025-08-01")
+		(rev "V0.1")
+		(company "telelmetry.digital s.r.o.")
+	)
 	(no_connect
 		(at 85.09 125.73)
@@
 		(dnp no)
 		(fields_autoplaced yes)
-		(property "Reference" "U2"
+		(property "Reference" "U3"
 			(at 100.33 58.3498 0)
 			(effects
@@
 				(path "/a02e5dd1-80da-4253-b87a-c8707aa3e0b0/831bc4de-0744-4eeb-b882-33b45fc786ec"
 					(reference "U7")
-					(unit 1)
-				)
-				(path "/a02e5dd1-80da-4253-b87a-c8707aa3e0b0/9eb8d42e-6154-4c2e-a139-649ab80f1930"
-					(reference "U2")
 					(unit 1)
 				)
@@
 		(on_board yes)
 		(dnp no)
-		(property "Reference" "#PWR07"
+		(property "Reference" "#PWR08"
 			(at 58.42 50.8 0)
 			(effects
@@
 				(path "/a02e5dd1-80da-4253-b87a-c8707aa3e0b0/831bc4de-0744-4eeb-b882-33b45fc786ec"
 					(reference "#PWR012")
-					(unit 1)
-				)
-				(path "/a02e5dd1-80da-4253-b87a-c8707aa3e0b0/9eb8d42e-6154-4c2e-a139-649ab80f1930"
-					(reference "#PWR07")
 					(unit 1)
 				)
@@
 		(on_board yes)
 		(dnp no)
-		(property "Reference" "#PWR01"
+		(property "Reference" "#PWR02"
 			(at 45.72 50.8 0)
 			(effects
@@
 				(path "/a02e5dd1-80da-4253-b87a-c8707aa3e0b0/831bc4de-0744-4eeb-b882-33b45fc786ec"
 					(reference "#PWR06")
-					(unit 1)
-				)
-				(path "/a02e5dd1-80da-4253-b87a-c8707aa3e0b0/9eb8d42e-6154-4c2e-a139-649ab80f1930"
-					(reference "#PWR01")
 					(unit 1)
 				)
@@
 		(dnp no)
 		(fields_autoplaced yes)
-		(property "Reference" "C13"
+		(property "Reference" "C14"
 			(at 62.23 38.0999 0)
 			(effects
@@
 				(path "/a02e5dd1-80da-4253-b87a-c8707aa3e0b0/831bc4de-0744-4eeb-b882-33b45fc786ec"
 					(reference "C18")
-					(unit 1)
-				)
-				(path "/a02e5dd1-80da-4253-b87a-c8707aa3e0b0/9eb8d42e-6154-4c2e-a139-649ab80f1930"
-					(reference "C13")
 					(unit 1)
 				)
@@
 		(on_board yes)
 		(dnp no)
-		(property "Reference" "C1"
+		(property "Reference" "C2"
 			(at 49.53 57.1499 0)
 			(effects
@@
 				(path "/a02e5dd1-80da-4253-b87a-c8707aa3e0b0/831bc4de-0744-4eeb-b882-33b45fc786ec"
 					(reference "C6")
-					(unit 1)
-				)
-				(path "/a02e5dd1-80da-4253-b87a-c8707aa3e0b0/9eb8d42e-6154-4c2e-a139-649ab80f1930"
-					(reference "C1")
 					(unit 1)
 				)
@@
 		(dnp no)
 		(fields_autoplaced yes)
-		(property "Reference" "C7"
+		(property "Reference" "C8"
 			(at 49.53 38.0999 0)
 			(effects
@@
 					(unit 1)
 				)
-				(path "/a02e5dd1-80da-4253-b87a-c8707aa3e0b0/9eb8d42e-6154-4c2e-a139-649ab80f1930"
-					(reference "C7")
-					(unit 1)
-				)

Commit message: update
Parts:
- renumbered C8 to C1, C14 to C3, U3 to U2
Changed lines of the file:
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@@
 		(dnp no)
 		(fields_autoplaced yes)
-		(property "Reference" "U3"
+		(property "Reference" "U2"
 			(at 100.33 58.3498 0)
 			(effects
@@
 				)
 				(path "/a02e5dd1-80da-4253-b87a-c8707aa3e0b0/4927e2a7-a4c2-4e52-af67-49600773c73d"
-					(reference "U5")
+					(reference "U4")
+					(unit 1)
+				)
+				(path "/a02e5dd1-80da-4253-b87a-c8707aa3e0b0/821b2e97-406d-4e86-b34c-70394fee7de3"
+					(reference "U2")
 					(unit 1)
 				)
@@
 				)
 				(path "/a02e5dd1-80da-4253-b87a-c8707aa3e0b0/bc306ebc-9231-4e41-974d-f78f75c244a9"
-					(reference "U4")
+					(reference "U5")
 					(unit 1)
 				)
@@
 		(on_board yes)
 		(dnp no)
-		(property "Reference" "#PWR08"
+		(property "Reference" "#PWR02"
 			(at 58.42 50.8 0)
 			(effects
@@
 			(project "pnp32_mainboard"
 				(path "/a02e5dd1-80da-4253-b87a-c8707aa3e0b0/36c8ee69-d46e-4392-9648-7ffe454aa773"
-					(reference "#PWR011")
+					(reference "#PWR010")
 					(unit 1)
 				)
 				(path "/a02e5dd1-80da-4253-b87a-c8707aa3e0b0/4927e2a7-a4c2-4e52-af67-49600773c73d"
-					(reference "#PWR010")
+					(reference "#PWR06")
+					(unit 1)
+				)
+				(path "/a02e5dd1-80da-4253-b87a-c8707aa3e0b0/821b2e97-406d-4e86-b34c-70394fee7de3"
+					(reference "#PWR02")
 					(unit 1)
 				)
@@
 				)
 				(path "/a02e5dd1-80da-4253-b87a-c8707aa3e0b0/a54d937e-12a5-4dff-8c5d-763d1b46ce81"
+					(reference "#PWR04")
+					(unit 1)
+				)
+				(path "/a02e5dd1-80da-4253-b87a-c8707aa3e0b0/bc306ebc-9231-4e41-974d-f78f75c244a9"
 					(reference "#PWR08")
-					(unit 1)
-				)
-				(path "/a02e5dd1-80da-4253-b87a-c8707aa3e0b0/bc306ebc-9231-4e41-974d-f78f75c244a9"
-					(reference "#PWR09")
 					(unit 1)
 				)
@@
 		(on_board yes)
 		(dnp no)
-		(property "Reference" "#PWR02"
+		(property "Reference" "#PWR01"
 			(at 45.72 50.8 0)
 			(effects
@@
 			(project ""
 				(path "/a02e5dd1-80da-4253-b87a-c8707aa3e0b0/36c8ee69-d46e-4392-9648-7ffe454aa773"
+					(reference "#PWR09")
+					(unit 1)
+				)
+				(path "/a02e5dd1-80da-4253-b87a-c8707aa3e0b0/4927e2a7-a4c2-4e52-af67-49600773c73d"
 					(reference "#PWR05")
 					(unit 1)
 				)
-				(path "/a02e5dd1-80da-4253-b87a-c8707aa3e0b0/4927e2a7-a4c2-4e52-af67-49600773c73d"
-					(reference "#PWR04")
+				(path "/a02e5dd1-80da-4253-b87a-c8707aa3e0b0/821b2e97-406d-4e86-b34c-70394fee7de3"
+					(reference "#PWR01")
 					(unit 1)
 				)
 				(path "/a02e5dd1-80da-4253-b87a-c8707aa3e0b0/831bc4de-0744-4eeb-b882-33b45fc786ec"
-					(reference "#PWR06")
+					(reference "#PWR011")
 					(unit 1)
 				)
 				(path "/a02e5dd1-80da-4253-b87a-c8707aa3e0b0/a54d937e-12a5-4dff-8c5d-763d1b46ce81"
-					(reference "#PWR02")
+					(reference "#PWR03")
 					(unit 1)
 				)
 				(path "/a02e5dd1-80da-4253-b87a-c8707aa3e0b0/bc306ebc-9231-4e41-974d-f78f75c244a9"
-					(reference "#PWR03")
+					(reference "#PWR07")
 					(unit 1)
 				)
@@
 		(dnp no)
 		(fields_autoplaced yes)
-		(property "Reference" "C14"
+		(property "Reference" "C3"
 			(at 62.23 38.0999 0)
 			(effects
@@
 			(project ""
 				(path "/a02e5dd1-80da-4253-b87a-c8707aa3e0b0/36c8ee69-d46e-4392-9648-7ffe454aa773"
-					(reference "C17")
+					(reference "C15")
 					(unit 1)
 				)
 				(path "/a02e5dd1-80da-4253-b87a-c8707aa3e0b0/4927e2a7-a4c2-4e52-af67-49600773c73d"
-					(reference "C16")
+					(reference "C9")
+					(unit 1)
+				)
+				(path "/a02e5dd1-80da-4253-b87a-c8707aa3e0b0/821b2e97-406d-4e86-b34c-70394fee7de3"
+					(reference "C3")
 					(unit 1)
 				)
@@
 				)
 				(path "/a02e5dd1-80da-4253-b87a-c8707aa3e0b0/a54d937e-12a5-4dff-8c5d-763d1b46ce81"
-					(reference "C14")
+					(reference "C6")
 					(unit 1)
 				)
 				(path "/a02e5dd1-80da-4253-b87a-c8707aa3e0b0/bc306ebc-9231-4e41-974d-f78f75c244a9"
-					(reference "C15")
+					(reference "C12")
 					(unit 1)
 				)
@@
 			(project ""
 				(path "/a02e5dd1-80da-4253-b87a-c8707aa3e0b0/36c8ee69-d46e-4392-9648-7ffe454aa773"
+					(reference "C14")
+					(unit 1)
+				)
+				(path "/a02e5dd1-80da-4253-b87a-c8707aa3e0b0/4927e2a7-a4c2-4e52-af67-49600773c73d"
+					(reference "C8")
+					(unit 1)
+				)
+				(path "/a02e5dd1-80da-4253-b87a-c8707aa3e0b0/821b2e97-406d-4e86-b34c-70394fee7de3"
+					(reference "C2")
+					(unit 1)
+				)
+				(path "/a02e5dd1-80da-4253-b87a-c8707aa3e0b0/831bc4de-0744-4eeb-b882-33b45fc786ec"
+					(reference "C17")
+					(unit 1)
+				)
+				(path "/a02e5dd1-80da-4253-b87a-c8707aa3e0b0/a54d937e-12a5-4dff-8c5d-763d1b46ce81"
 					(reference "C5")
 					(unit 1)
 				)
-				(path "/a02e5dd1-80da-4253-b87a-c8707aa3e0b0/4927e2a7-a4c2-4e52-af67-49600773c73d"
-					(reference "C4")
-					(unit 1)
-				)
-				(path "/a02e5dd1-80da-4253-b87a-c8707aa3e0b0/831bc4de-0744-4eeb-b882-33b45fc786ec"
-					(reference "C6")
-					(unit 1)
-				)
-				(path "/a02e5dd1-80da-4253-b87a-c8707aa3e0b0/a54d937e-12a5-4dff-8c5d-763d1b46ce81"
-					(reference "C2")
-					(unit 1)
-				)
 				(path "/a02e5dd1-80da-4253-b87a-c8707aa3e0b0/bc306ebc-9231-4e41-974d-f78f75c244a9"
-					(reference "C3")
+					(reference "C11")
 					(unit 1)
 				)
@@
 		(dnp no)
 		(fields_autoplaced yes)
-		(property "Reference" "C8"
+		(property "Reference" "C1"
 			(at 49.53 38.0999 0)
 			(effects
@@
 			(project ""
 				(path "/a02e5dd1-80da-4253-b87a-c8707aa3e0b0/36c8ee69-d46e-4392-9648-7ffe454aa773"
-					(reference "C11")
+					(reference "C13")
 					(unit 1)
 				)
 				(path "/a02e5dd1-80da-4253-b87a-c8707aa3e0b0/4927e2a7-a4c2-4e52-af67-49600773c73d"
+					(reference "C7")
+					(unit 1)
+				)
+				(path "/a02e5dd1-80da-4253-b87a-c8707aa3e0b0/821b2e97-406d-4e86-b34c-70394fee7de3"
+					(reference "C1")
+					(unit 1)
+				)
+				(path "/a02e5dd1-80da-4253-b87a-c8707aa3e0b0/831bc4de-0744-4eeb-b882-33b45fc786ec"
+					(reference "C16")
+					(unit 1)
+				)
+				(path "/a02e5dd1-80da-4253-b87a-c8707aa3e0b0/a54d937e-12a5-4dff-8c5d-763d1b46ce81"
+					(reference "C4")
+					(unit 1)
+				)
+				(path "/a02e5dd1-80da-4253-b87a-c8707aa3e0b0/bc306ebc-9231-4e41-974d-f78f75c244a9"
 					(reference "C10")
 					(unit 1)
 				)
-				(path "/a02e5dd1-80da-4253-b87a-c8707aa3e0b0/831bc4de-0744-4eeb-b882-33b45fc786ec"
-					(reference "C12")
-					(unit 1)
-				)
-				(path "/a02e5dd1-80da-4253-b87a-c8707aa3e0b0/a54d937e-12a5-4dff-8c5d-763d1b46ce81"
-					(reference "C8")
-					(unit 1)
-				)
-				(path "/a02e5dd1-80da-4253-b87a-c8707aa3e0b0/bc306ebc-9231-4e41-974d-f78f75c244a9"
-					(reference "C9")
-					(unit 1)
-				)

Commit message: update
Parts:
- added C23, C25, C26, C27: 470p, Capacitor_SMD:C_0805_2012Metric, symbol Device:C_Small
- added C28, C29, C32, C33, C34: 100n, Capacitor_SMD:C_0805_2012Metric, symbol Device:C_Small
- added C30: 100u, Capacitor_SMD:CP_Elec_6.3x7.7, symbol Device:C_Polarized_Small
- added C31: 10u, Capacitor_SMD:C_0805_2012Metric, symbol Device:C_Small
- added J2: MOTOR, Connector_JST:JST_PH_B4B-PH-SM4-TB_1x04-1MP_P2.00mm_Vertical, symbol Connector_Generic_MountingPin:Conn_01x04_MountingPin
- added L3, L4, L5, L6: L_Ferrite, Inductor_SMD:L_0805_2012Metric, symbol Device:L_Ferrite
- added R16, R17: 120m, Resistor_SMD:R_2512_6332Metric, symbol Device:R_Small
- added TP6, TP7, TP8, TP9: TestPoint, TestPoint:TestPoint_Pad_D2.0mm, symbol Connector:TestPoint
- renumbered C1 to C21, C3 to C22, C2 to C24, U2 to U8
Connections:
- net GND: now also C23.1, C25.2, C26.1, C27.2, C28.1, C29.1, C30.2, C31.1, C32.1, C33.1, C34.1, J2.MP (MountPin), R16.2, R17.2
- net at U8.15 (OB1): now also L5.1
- net at U8.17 (BRB): now also C28.2, R16.1
- net at U8.19 (OB2): now also L6.1
- net at U8.42 (OA2): now also L4.1
- net at U8.44 (BRA): now also C29.2, R17.1
- net at U8.46 (OA1): now also L3.1
- new net +3.3V: C34.2
- new net A1: C23.2, J2.3 (Pin_3), L3.2, TP6.1
- new net A2: C25.1, J2.4 (Pin_4), L4.2, TP7.1
- new net B1: C26.2, J2.2 (Pin_2), L5.2, TP8.1
- new net B2: C27.1, J2.1 (Pin_1), L6.2, TP9.1
- new net VDC: C30.1, C31.2, C32.2, C33.2
Other:
- note added: "Place close to VCC_IO"
