File: HARDWARE/pnp32_controller/pnp32_mainboard/mosfet.kicad_sch (KiCad schematic)
At the start: 7 parts, among them J8 FET, Q1 AO3400A, U14 PESD24BS3

Commit message: update_PSU
Parts:
- removed J8: FET, Connector_JST:JST_PH_B2B-PH-SM4-TB_1x02-1MP_P2.00mm_Vertical, symbol Connector_Generic_MountingPin:Conn_01x02_MountingPin
- added J9: Conn_01x02_Pin, fab_CON:WE_620302124022, symbol fab_CON:WE_620302124022
- renumbered D9 to D13, Q1 to Q2, R28 to R32, R29 to R33
Connections:
- net VDC: now also J9.1 (Pin_1)
- net at D13.2 (A), Q2.3 (D), TP30.1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: now also J9.2 (Pin_2)
