File: HARDWARE/pnp32_controller/pnp32_mainboard/pnp32_mainboard.kicad_pcb (KiCad board)
At the start: 2 copper layers, 80 x 40 mm, 4 parts, among them U1 ESP32-PICO-V3, U2 TMC5130A-TA, U3 TMC5130A-TA, U4 TMC5130A-TA

Commit message: update
Parts:
- added U5: TMC5130A-TA, Package_QFP:TQFP-48-1EP_7x7mm_P0.5mm_EP5x5mm_ThermalVias, F.Cu at (156.5, 90.3)
- added U6: TMC5130A-TA, Package_QFP:TQFP-48-1EP_7x7mm_P0.5mm_EP5x5mm_ThermalVias, F.Cu at (171.5, 90.3)
- added U7: TMC5130A-TA, Package_QFP:TQFP-48-1EP_7x7mm_P0.5mm_EP5x5mm_ThermalVias, F.Cu at (186.6, 90.3)
- moved U4 40.5 mm to (141.5, 90.3)
- moved U3 40.0 mm to (127.0, 90.3)
- moved U2 39.3 mm to (111.5, 90.3)
- moved U1 20.2 mm to (110.7, 109.6)
Connections:
- U1 pad 14: unconnected-(U1-GPIO25/ADC2_CH8/DAC_1-Pad14) -> /B-driver/SPI_CS
- U1 pad 15: unconnected-(U1-GPIO26/ADC2_CH9/DAC_2-Pad15) -> /C-driver/SPI_CS
- U1 pad 22: unconnected-(U1-GPIO2/ADC2_CH2-Pad22) -> /A-driver/SPI_MISO
- U1 pad 24: unconnected-(U1-GPIO4/ADC2_CH0-Pad24) -> /A-driver/SPI_MOSI
- U1 pad 27: unconnected-(U1-GPIO20-Pad27) -> /CPU/SPI_CS_Y
- U1 pad 31: unconnected-(U1-SD_CLK/GPIO6-Pad31) -> /CPU/I2C_SDA
- U1 pad 32: unconnected-(U1-SD_DATA_0/GPIO7-Pad32) -> /CPU/I2C_SCL
- U1 pad 34: unconnected-(U1-GPIO5-Pad34) -> /A-driver/SPI_CLK
- U1 pad 38: unconnected-(U1-GPIO19-Pad38) -> /CPU/SPI_CS_X
- U1 pad 39: unconnected-(U1-GPIO22-Pad39) -> /A-driver/SPI_CS
- U1 pad 42: unconnected-(U1-GPIO21-Pad42) -> /CPU/SPI_CS_Z
- U2 pad 3: SPI_CS -> /CPU/SPI_CS_X
- U2 pad 4: SPI_CLK -> /A-driver/SPI_CLK
- U2 pad 5: SPI_MOSI -> /A-driver/SPI_MOSI
- U2 pad 7: SPI_MISO -> /A-driver/SPI_MISO
- U3 pad 3: SPI_CS -> /CPU/SPI_CS_Y
- U3 pad 4: SPI_CLK -> /A-driver/SPI_CLK
- U3 pad 5: SPI_MOSI -> /A-driver/SPI_MOSI
- U3 pad 7: SPI_MISO -> /A-driver/SPI_MISO
- U4 pad 3: SPI_CS -> /A-driver/SPI_CS
- U4 pad 4: SPI_CLK -> /A-driver/SPI_CLK
- U4 pad 5: SPI_MOSI -> /A-driver/SPI_MOSI
- U4 pad 7: SPI_MISO -> /A-driver/SPI_MISO
Other:
- board size 80 x 40 mm -> 100 x 40 mm

Commit message: update_firmware
Other:
- board text added: "https://github.com/palo-krnac/pnp32"
Changed lines of the file:
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@@
 		(layer "Edge.Cuts")
+	)
+	(gr_text "https://github.com/palo-krnac/pnp32"
+		(at 153.31 119.38 0)
+		(layer "F.Cu")
+		(effects
+			(font
+				(size 1.5 1.5)
+				(thickness 0.3)
+				(bold yes)
+			)
+			(justify left bottom)
+		)
 	)
 	(embedded_fonts no)

Commit message: update
Parts:
- added C1: 22nF/0805, fab_C:C_0805, F.Cu at (106.6, 85.4)
- added C10: 4.7uF, fab_C:C_0603, F.Cu at (129.7, 69.4)
- added C11: 4.7uF, fab_C:C_0603, F.Cu at (129.7, 62.4)
- added C12: 4.7uF, fab_C:C_0603, F.Cu at (135.7, 62.4)
- added C13: 470nF, fab_C:C_0603, F.Cu at (141.7, 64.9)
- added C14: 470nF, fab_C:C_0603, F.Cu at (135.7, 71.9)
- added C15: 470nF, fab_C:C_0603, F.Cu at (141.7, 71.9)
- added C16: 470nF, fab_C:C_0603, F.Cu at (129.7, 71.9)
- added C17: 470nF, fab_C:C_0603, F.Cu at (129.7, 64.9)
- added C18: 470nF, fab_C:C_0603, F.Cu at (135.7, 64.9)
- added C2: 22nF/0805, fab_C:C_0805, F.Cu at (165.1, 67.8)
- added C3: 22nF/0805, fab_C:C_0805, F.Cu at (166.1, 84.5)
- added C4: 22nF/0805, fab_C:C_0805, F.Cu at (165.1, 62.9)
- added C5: 22nF/0805, fab_C:C_0805, F.Cu at (158.7, 62.9)
- added C6: 22nF/0805, fab_C:C_0805, F.Cu at (158.7, 67.8)
- added C7: 4.7uF, fab_C:C_0603, F.Cu at (141.7, 62.4)
- added C8: 4.7uF, fab_C:C_0603, F.Cu at (135.7, 69.4)
- added C9: 4.7uF, fab_C:C_0603, F.Cu at (141.7, 69.4)
- U2, U3, U4, U5, U6, U7: footprint Package_QFP:TQFP-48-1EP_7x7mm_P0.5mm_EP5x5mm_ThermalVias -> fab_U:TQFP-48-1EP_7x7mm_P0.5mm_EP5x5mm_ThermalVias
- turned U1 to 90 degrees
- turned U2 to 90 degrees
- turned U3 to 90 degrees
- turned U4 to 90 degrees
- turned U5 to 90 degrees
- turned U6 to 90 degrees
- turned U7 to 90 degrees
Connections:
- U2 pad 33: unconnected-(U2-5VOUT-Pad33) -> Net-(U2-5VOUT)
- U2 pad 34: unconnected-(U2-VCC-Pad34) -> Net-(U2-VCC)
- U2 pad 35: unconnected-(U2-CP0-Pad35) -> /X-driver/CPO
- U2 pad 37: unconnected-(U2-CPI-Pad37) -> /X-driver/CPI
- U3 pad 33: unconnected-(U3-5VOUT-Pad33) -> Net-(U3-5VOUT)
- U3 pad 34: unconnected-(U3-VCC-Pad34) -> Net-(U3-VCC)
- U3 pad 35: unconnected-(U3-CP0-Pad35) -> /Y-driver/CPO
- U3 pad 37: unconnected-(U3-CPI-Pad37) -> /Y-driver/CPI
- U4 pad 33: unconnected-(U4-5VOUT-Pad33) -> Net-(U4-5VOUT)
- U4 pad 34: unconnected-(U4-VCC-Pad34) -> Net-(U4-VCC)
- U4 pad 35: unconnected-(U4-CP0-Pad35) -> /A-driver/CPO
- U4 pad 37: unconnected-(U4-CPI-Pad37) -> /A-driver/CPI
- U5 pad 33: unconnected-(U5-5VOUT-Pad33) -> Net-(U5-5VOUT)
- U5 pad 34: unconnected-(U5-VCC-Pad34) -> Net-(U5-VCC)
- U5 pad 35: unconnected-(U5-CP0-Pad35) -> /Z-driver/CPO
- U5 pad 37: unconnected-(U5-CPI-Pad37) -> /Z-driver/CPI
- U6 pad 33: unconnected-(U6-5VOUT-Pad33) -> Net-(U6-5VOUT)
- U6 pad 34: unconnected-(U6-VCC-Pad34) -> Net-(U6-VCC)
- U6 pad 35: unconnected-(U6-CP0-Pad35) -> /B-driver/CPO
- U6 pad 37: unconnected-(U6-CPI-Pad37) -> /B-driver/CPI
- U7 pad 33: unconnected-(U7-5VOUT-Pad33) -> Net-(U7-5VOUT)
- U7 pad 34: unconnected-(U7-VCC-Pad34) -> Net-(U7-VCC)
- U7 pad 35: unconnected-(U7-CP0-Pad35) -> /C-driver/CPO
- U7 pad 37: unconnected-(U7-CPI-Pad37) -> /C-driver/CPI
Routing:
- net /A-driver/SPI_MOSI: track 0.00 -> 93.0 mm, vias 0 -> 10
- net /A-driver/SPI_MISO: track 0.00 -> 88.9 mm
- net /A-driver/SPI_CLK: track 0.00 -> 78.0 mm
- net /X-driver/CPO: track 0.00 -> 2.96 mm
- net /X-driver/CPI: track 0.00 -> 2.70 mm
Other:
- board text added: "pnp32"

Commit message: update
Parts:
- added C1: 4.7uF, fab_C:C_0603, F.Cu at (93.5, 84.6)
- added C2: 22nF/0805, fab_C:C_0805, F.Cu at (82.3, 96.2)
- added C3: 470nF, fab_C:C_0603, F.Cu at (93.5, 87.2)
- moved C10 44.7 mm to (137.7, 114.0)
- moved C13 44.7 mm to (125.7, 106.9)
- moved C16 44.7 mm to (131.7, 106.9)
- moved C4 44.7 mm to (131.7, 114.0)
- moved C5 44.7 mm to (161.1, 112.4)
- moved C7 44.7 mm to (125.7, 114.0)
- moved C7 44.7 mm to (137.7, 106.9)
- moved C12 44.7 mm to (137.7, 116.5)
- moved C13 44.7 mm to (137.7, 109.4)
- moved C15 44.7 mm to (125.7, 109.4)
- moved C18 44.7 mm to (131.7, 109.4)
- moved C6 44.7 mm to (131.7, 116.5)
- moved C9 44.7 mm to (125.7, 116.5)
- moved C11 29.3 mm to (136.8, 85.5), turned to -90 degrees
- moved C17 29.2 mm to (181.9, 85.5), turned to -90 degrees
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- renumbered C9 to C10, C3 to C11, C15 to C12, C11 to C13, C5 to C14, C17 to C15, C12 to C16, C6 to C17, C1 to C2, C8 to C4, C2 to C5, C14 to C6, C10 to C7, C4 to C8, C16 to C9, U5 to U4, U4 to U5
Connections:
- U1 pad 1: Net-(U1-VDDA-Pad1) -> +3.3V
- U1 pad 10: unconnected-(U1-VDET_1/GPIO34/ADC1_CH6-Pad10) -> /CPU/VAC1
- U1 pad 11: unconnected-(U1-VDET_2/GPIO35/ADC1_CH7-Pad11) -> /CPU/VAC2
- U1 pad 12: unconnected-(U1-32K_XP/GPIO32/ADC1_CH4-Pad12) -> /CPU/ENABLE
- U1 pad 13: unconnected-(U1-32K_XN/GPIO33/ADC1_CH5-Pad13) -> /CPU/E-STOP
- U1 pad 17: unconnected-(U1-MTMS/GPIO14/ADC2_CH6-Pad17) -> /CPU/PIN_RD
- U1 pad 18: unconnected-(U1-MTDI/GPIO12/ADC2_CH5-Pad18) -> /CPU/RS485_A
- U1 pad 19: unconnected-(U1-VDD3P3_RTC-Pad19) -> +3.3V
- U1 pad 20: unconnected-(U1-MTCK/GPIO13/ADC2_CH4-Pad20) -> /CPU/RS485_B
- U1 pad 21: unconnected-(U1-MTDO/GPIO15/ADC2_CH3-Pad21) -> /CPU/PIN_WR
- U1 pad 26: unconnected-(U1-VDD_SDIO-Pad26) -> +3.3V
- U1 pad 3: Net-(U1-VDD3P3-Pad3) -> +3.3V
- U1 pad 33: unconnected-(U1-SD_DATA_1/GPIO8-Pad33) -> /CPU/WLED
- U1 pad 37: unconnected-(U1-VDD3P3_CPU-Pad37) -> +3.3V
- U1 pad 4: Net-(U1-VDD3P3-Pad3) -> +3.3V
- U1 pad 43: Net-(U1-VDDA-Pad1) -> +3.3V
- U1 pad 46: Net-(U1-VDDA-Pad1) -> +3.3V
- U1 pad 49: unconnected-(U1-GND-Pad49) -> GND
- U1 pad 5: unconnected-(U1-SENSOR_VP/GPIO36/ADC1_CH0-Pad5) -> /CPU/VAC_PUMP
- U1 pad 6: unconnected-(U1-SENSOR_CAPP/GPIO37/ADC1_CH1-Pad6) -> /CPU/AIR1
- U1 pad 7: unconnected-(U1-SENSOR_CAPN/GPIO38/ADC1_CH2-Pad7) -> /CPU/AIR2
- U1 pad 8: unconnected-(U1-SENSOR_VN/GPIO39/ADC1_CH3-Pad8) -> /CPU/AIR_PUMP
Routing:
- net /A-driver/SPI_CLK: track 78.0 -> 83.2 mm, vias 0 -> 2

Commit message: update
Parts:
- added BZ1: Buzzer, Buzzer_Beeper:MagneticBuzzer_CUI_CMT-8504-100-SMT, F.Cu at (212.4, 113.3)
- added C100: 100u, Capacitor_SMD:CP_Elec_6.3x7.7, F.Cu at (25.0, 140.0)
- added C101: 10u, Capacitor_SMD:C_0805_2012Metric, F.Cu at (25.0, 143.0)
- added C102: 100n, Capacitor_SMD:C_0805_2012Metric, F.Cu at (25.0, 146.0)
- added C103: 100n, Capacitor_SMD:C_0805_2012Metric, F.Cu at (142.0, 150.0)
- added C104: 100n, Capacitor_SMD:C_0805_2012Metric, F.Cu at (142.0, 153.0)
- added C19: 100n, Capacitor_SMD:C_0805_2012Metric, F.Cu at (68.8, 154.3)
- added C20: 100n, Capacitor_SMD:C_0805_2012Metric, F.Cu at (68.8, 156.8)
- added C21: 4.7uF, fab_C:C_0603, F.Cu at (47.3, 143.5)
- added C22: 470nF, fab_C:C_0603, F.Cu at (56.2, 153.3)
- added C23: 470p, Capacitor_SMD:C_0805_2012Metric, F.Cu at (47.3, 146.5)
- added C24: 22nF/0805, fab_C:C_0805, F.Cu at (47.3, 149.5)
- added C25: 470p, Capacitor_SMD:C_0805_2012Metric, F.Cu at (47.3, 152.6)
- added C26: 470p, Capacitor_SMD:C_0805_2012Metric, F.Cu at (47.3, 155.6)
- added C27: 470p, Capacitor_SMD:C_0805_2012Metric, F.Cu at (51.8, 143.5)
- added C28: 100n, Capacitor_SMD:C_0805_2012Metric, F.Cu at (64.8, 136.5)
- added C29: 100n, Capacitor_SMD:C_0805_2012Metric, F.Cu at (51.8, 146.5)
- added C30: 100u, Capacitor_SMD:CP_Elec_6.3x7.7, F.Cu at (51.8, 149.5)
- added C31: 10u, Capacitor_SMD:C_0805_2012Metric, F.Cu at (51.8, 152.6)
- added C32: 100n, Capacitor_SMD:C_0805_2012Metric, F.Cu at (51.8, 155.6)
- added C33: 100n, Capacitor_SMD:C_0805_2012Metric, F.Cu at (97.0, 154.3)
- added C34: 100n, Capacitor_SMD:C_0805_2012Metric, F.Cu at (97.0, 156.8)
- added C35: 4.7uF, fab_C:C_0603, F.Cu at (75.5, 143.5)
- added C36: 470nF, fab_C:C_0603, F.Cu at (84.5, 153.3)
- added C37: 470p, Capacitor_SMD:C_0805_2012Metric, F.Cu at (75.5, 146.5)
- added C38: 22nF/0805, fab_C:C_0805, F.Cu at (75.5, 149.5)
- added C39: 470p, Capacitor_SMD:C_0805_2012Metric, F.Cu at (75.5, 152.6)
- added C40: 470p, Capacitor_SMD:C_0805_2012Metric, F.Cu at (75.5, 155.6)
- added C41: 470p, Capacitor_SMD:C_0805_2012Metric, F.Cu at (80.0, 143.5)
- added C42: 100n, Capacitor_SMD:C_0805_2012Metric, F.Cu at (93.0, 136.5)
- added C43: 100n, Capacitor_SMD:C_0805_2012Metric, F.Cu at (80.0, 146.5)
- added C44: 100u, Capacitor_SMD:CP_Elec_6.3x7.7, F.Cu at (80.0, 149.5)
- added C45: 10u, Capacitor_SMD:C_0805_2012Metric, F.Cu at (80.0, 152.6)
- added C46: 100n, Capacitor_SMD:C_0805_2012Metric, F.Cu at (80.0, 155.6)
- added C47: 100n, Capacitor_SMD:C_0805_2012Metric, F.Cu at (100.0, 123.5)
- added C48: 100n, Capacitor_SMD:C_0805_2012Metric, F.Cu at (100.0, 126.0)
- added C49: 4.7uF, fab_C:C_0603, F.Cu at (80.9, 102.9)
- added C50: 470nF, fab_C:C_0603, F.Cu at (100.3, 128.8)
- added C51: 470p, Capacitor_SMD:C_0805_2012Metric, F.Cu at (80.9, 105.9)
- added C52: 22nF/0805, fab_C:C_0805, F.Cu at (80.9, 108.9)
- added C53: 470p, Capacitor_SMD:C_0805_2012Metric, F.Cu at (80.9, 111.9)
- added C54: 470p, Capacitor_SMD:C_0805_2012Metric, F.Cu at (80.9, 114.9)
- added C55: 470p, Capacitor_SMD:C_0805_2012Metric, F.Cu at (85.4, 102.9)
- added C56: 100n, Capacitor_SMD:C_0805_2012Metric, F.Cu at (92.8, 126.3)
- added C57: 100n, Capacitor_SMD:C_0805_2012Metric, F.Cu at (85.4, 105.9)
- added C58: 100u, Capacitor_SMD:CP_Elec_6.3x7.7, F.Cu at (85.4, 108.9)
- added C59: 10u, Capacitor_SMD:C_0805_2012Metric, F.Cu at (85.4, 111.9)
- added C60: 100n, Capacitor_SMD:C_0805_2012Metric, F.Cu at (85.4, 114.9)
- added C61: 100n, Capacitor_SMD:C_0805_2012Metric, F.Cu at (39.7, 185.7)
- added C62: 100n, Capacitor_SMD:C_0805_2012Metric, F.Cu at (39.7, 188.2)
- added C63: 4.7uF, fab_C:C_0603, F.Cu at (20.5, 165.0)
- added C64: 470nF, fab_C:C_0603, F.Cu at (39.9, 190.9)
- added C65: 470p, Capacitor_SMD:C_0805_2012Metric, F.Cu at (20.5, 168.0)
- added C66: 22nF/0805, fab_C:C_0805, F.Cu at (20.5, 171.0)
- added C67: 470p, Capacitor_SMD:C_0805_2012Metric, F.Cu at (20.5, 174.1)
- added C68: 470p, Capacitor_SMD:C_0805_2012Metric, F.Cu at (20.5, 177.1)
- added C69: 470p, Capacitor_SMD:C_0805_2012Metric, F.Cu at (25.0, 165.0)
- added C70: 100n, Capacitor_SMD:C_0805_2012Metric, F.Cu at (32.4, 188.5)
- added C71: 100n, Capacitor_SMD:C_0805_2012Metric, F.Cu at (25.0, 168.0)
- added C72: 100u, Capacitor_SMD:CP_Elec_6.3x7.7, F.Cu at (25.0, 171.0)
- added C73: 10u, Capacitor_SMD:C_0805_2012Metric, F.Cu at (25.0, 174.1)
- added C74: 100n, Capacitor_SMD:C_0805_2012Metric, F.Cu at (25.0, 177.1)
- added C75: 100n, Capacitor_SMD:C_0805_2012Metric, F.Cu at (69.2, 123.5)
- added C76: 100n, Capacitor_SMD:C_0805_2012Metric, F.Cu at (69.2, 126.0)
- added C77: 4.7uF, fab_C:C_0603, F.Cu at (50.1, 102.9)
- added C78: 470nF, fab_C:C_0603, F.Cu at (69.4, 128.8)
- added C79: 470p, Capacitor_SMD:C_0805_2012Metric, F.Cu at (50.1, 105.9)
- added C80: 22nF/0805, fab_C:C_0805, F.Cu at (50.1, 108.9)
- added C81: 470p, Capacitor_SMD:C_0805_2012Metric, F.Cu at (50.1, 111.9)
- added C82: 470p, Capacitor_SMD:C_0805_2012Metric, F.Cu at (50.1, 114.9)
- added C83: 470p, Capacitor_SMD:C_0805_2012Metric, F.Cu at (54.5, 102.9)
- added C84: 100n, Capacitor_SMD:C_0805_2012Metric, F.Cu at (62.0, 126.3)
- added C85: 100n, Capacitor_SMD:C_0805_2012Metric, F.Cu at (54.5, 105.9)
- added C86: 100u, Capacitor_SMD:CP_Elec_6.3x7.7, F.Cu at (54.5, 108.9)
- added C87: 10u, Capacitor_SMD:C_0805_2012Metric, F.Cu at (54.5, 111.9)
- added C88: 100n, Capacitor_SMD:C_0805_2012Metric, F.Cu at (54.5, 114.9)
- added C89: 100n, Capacitor_SMD:C_0805_2012Metric, F.Cu at (39.7, 154.6)
- added C90: 100n, Capacitor_SMD:C_0805_2012Metric, F.Cu at (39.7, 157.1)
- added C91: 4.7uF, fab_C:C_0603, F.Cu at (20.5, 134.0)
- added C92: 470nF, fab_C:C_0603, F.Cu at (39.9, 159.9)
- added C93: 470p, Capacitor_SMD:C_0805_2012Metric, F.Cu at (20.5, 137.0)
- added C94: 22nF/0805, fab_C:C_0805, F.Cu at (20.5, 140.0)
- added C95: 470p, Capacitor_SMD:C_0805_2012Metric, F.Cu at (20.5, 143.0)
- added C96: 470p, Capacitor_SMD:C_0805_2012Metric, F.Cu at (20.5, 146.0)
- added C97: 470p, Capacitor_SMD:C_0805_2012Metric, F.Cu at (25.0, 134.0)
- added C98: 100n, Capacitor_SMD:C_0805_2012Metric, F.Cu at (32.4, 157.4)
- added C99: 100n, Capacitor_SMD:C_0805_2012Metric, F.Cu at (25.0, 137.0)
- added D1: BZT52C16, Diode_SMD:D_SOD-123, F.Cu at (34.5, 111.2)
- added D10: SM4007, Diode_SMD:D_SOD-123F, F.Cu at (76.3, 184.0)
- added D11: SM4007, Diode_SMD:D_SOD-123F, F.Cu at (58.3, 184.0)
- added D12: SM4007, Diode_SMD:D_SOD-123F, F.Cu at (58.3, 167.8)
- added D13: SM4007, Diode_SMD:D_SOD-123F, F.Cu at (94.2, 167.8)
- added D14: SM4007, Diode_SMD:D_SOD-123F, F.Cu at (76.3, 167.8)
- added D15: SM4007, Diode_SMD:D_SOD-123F, F.Cu at (220.7, 109.3)
- added D16: SM4007, Diode_SMD:D_SOD-123F, F.Cu at (220.7, 112.7)
- added D17: LESD5D5.0CT1G, fab_D:SOD-523, F.Cu at (233.2, 133.9)
- added D18: LESD5D5.0CT1G, fab_D:SOD-523, F.Cu at (233.2, 118.4)
- added D19: LESD5D5.0CT1G, fab_D:SOD-523, F.Cu at (233.2, 149.4)
- added D2: BZT52C16, Diode_SMD:D_SOD-123, F.Cu at (34.5, 114.5)
- added D20: LESD5D5.0CT1G, fab_D:SOD-523, F.Cu at (247.7, 118.4)
- added D21: LESD5D5.0CT1G, fab_D:SOD-523, F.Cu at (247.7, 133.9)
- added D3: SMF28A, Diode_SMD:D_SMF, F.Cu at (34.5, 117.9)
- added D4: B560C, Diode_SMD:D_SMC, F.Cu at (19.7, 126.6)
- added D5: SS34, Diode_SMD:D_SMA, F.Cu at (35.6, 121.8)
- added D6: Green, LED_SMD:LED_0805_2012Metric, F.Cu at (39.6, 111.0)
- added D7: Green, LED_SMD:LED_0805_2012Metric, F.Cu at (39.6, 114.1)
- added D8: Green, LED_SMD:LED_0805_2012Metric, F.Cu at (39.6, 117.1)
- added D9: SM4007, Diode_SMD:D_SOD-123F, F.Cu at (94.2, 184.0)
- added F1: Fuse, Fuse:Fuseholder_Littelfuse_Nano2_154x, F.Cu at (20.4, 119.4)
- added FID1: Fiducial, Fiducial:Fiducial_1mm_Mask2mm, F.Cu at (215.7, 132.1)
- added FID2: Fiducial, Fiducial:Fiducial_1mm_Mask2mm, F.Cu at (215.7, 135.7)
- added FID3: Fiducial, Fiducial:Fiducial_1mm_Mask2mm, F.Cu at (215.7, 139.2)
- added FID4: Fiducial, Fiducial:Fiducial_1mm_Mask2mm, F.Cu at (215.7, 142.8)
- added H1: MountingHole_Pad, MountingHole:MountingHole_3.2mm_M3_DIN965_Pad, F.Cu at (210.4, 133.9)
- added H2: MountingHole_Pad, MountingHole:MountingHole_3.2mm_M3_DIN965_Pad, F.Cu at (210.4, 141.1)
- added H3: MountingHole_Pad, MountingHole:MountingHole_3.2mm_M3_DIN965_Pad, F.Cu at (210.4, 148.2)
- added H4: MountingHole_Pad, MountingHole:MountingHole_3.2mm_M3_DIN965_Pad, F.Cu at (210.4, 155.4)
- added J10: FET, Connector_JST:JST_PH_B2B-PH-SM4-TB_1x02-1MP_P2.00mm_Vertical, F.Cu at (50.3, 181.7)
- added J11: FET, Connector_JST:JST_PH_B2B-PH-SM4-TB_1x02-1MP_P2.00mm_Vertical, F.Cu at (50.3, 165.5)
- added J12: FET, Connector_JST:JST_PH_B2B-PH-SM4-TB_1x02-1MP_P2.00mm_Vertical, F.Cu at (86.2, 165.5)
- added J13: FET, Connector_JST:JST_PH_B2B-PH-SM4-TB_1x02-1MP_P2.00mm_Vertical, F.Cu at (68.3, 165.5)
- added J14: TOP_LIGHT, Connector_JST:JST_PH_B3B-PH-SM4-TB_1x03-1MP_P2.00mm_Vertical, F.Cu at (126.4, 169.1)
- added J15: TOP_LIGHT, Connector_JST:JST_PH_B3B-PH-SM4-TB_1x03-1MP_P2.00mm_Vertical, F.Cu at (126.4, 153.8)
- added J16: FAN, Connector_JST:JST_PH_B2B-PH-SM4-TB_1x02-1MP_P2.00mm_Vertical, F.Cu at (212.0, 124.1)
- added J17: TOP_LIGHT, Connector_JST:JST_PH_B3B-PH-SM4-TB_1x03-1MP_P2.00mm_Vertical, F.Cu at (234.8, 128.4)
- added J18: TOP_LIGHT, Connector_JST:JST_PH_B3B-PH-SM4-TB_1x03-1MP_P2.00mm_Vertical, F.Cu at (234.8, 112.9)
- added J19: TOP_LIGHT, Connector_JST:JST_PH_B3B-PH-SM4-TB_1x03-1MP_P2.00mm_Vertical, F.Cu at (234.8, 143.9)
- added J2: MOTOR, Connector_JST:JST_PH_B4B-PH-SM4-TB_1x04-1MP_P2.00mm_Vertical, F.Cu at (52.3, 137.7)
- added J20: TOP_LIGHT, Connector_JST:JST_PH_B3B-PH-SM4-TB_1x03-1MP_P2.00mm_Vertical, F.Cu at (249.2, 112.9)
- added J21: TOP_LIGHT, Connector_JST:JST_PH_B3B-PH-SM4-TB_1x03-1MP_P2.00mm_Vertical, F.Cu at (249.2, 128.4)
- added J3: MOTOR, Connector_JST:JST_PH_B4B-PH-SM4-TB_1x04-1MP_P2.00mm_Vertical, F.Cu at (80.5, 137.7)
- added J4: MOTOR, Connector_JST:JST_PH_B4B-PH-SM4-TB_1x04-1MP_P2.00mm_Vertical, F.Cu at (171.7, 70.7)
- added J5: MOTOR, Connector_JST:JST_PH_B4B-PH-SM4-TB_1x04-1MP_P2.00mm_Vertical, F.Cu at (34.4, 168.8)
- added J6: MOTOR, Connector_JST:JST_PH_B4B-PH-SM4-TB_1x04-1MP_P2.00mm_Vertical, F.Cu at (64.0, 106.7)
- added J7: MOTOR, Connector_JST:JST_PH_B4B-PH-SM4-TB_1x04-1MP_P2.00mm_Vertical, F.Cu at (34.4, 137.7)
- added J8: FET, Connector_JST:JST_PH_B2B-PH-SM4-TB_1x02-1MP_P2.00mm_Vertical, F.Cu at (86.2, 181.7)
- added J9: FET, Connector_JST:JST_PH_B2B-PH-SM4-TB_1x02-1MP_P2.00mm_Vertical, F.Cu at (68.3, 181.7)
- added L1: 2.2u, Inductor_SMD:L_Sunlord_MWSA0402S, F.Cu at (34.9, 127.0)
- added L10: L_Ferrite, Inductor_SMD:L_0805_2012Metric, F.Cu at (97.3, 151.6)
- added L11: L_Ferrite, Inductor_SMD:L_0805_2012Metric, F.Cu at (101.2, 112.3)
- added L12: L_Ferrite, Inductor_SMD:L_0805_2012Metric, F.Cu at (101.2, 115.0)
- added L13: L_Ferrite, Inductor_SMD:L_0805_2012Metric, F.Cu at (101.2, 117.8)
- added L14: L_Ferrite, Inductor_SMD:L_0805_2012Metric, F.Cu at (101.2, 120.5)
- added L15: L_Ferrite, Inductor_SMD:L_0805_2012Metric, F.Cu at (40.8, 174.4)
- added L16: L_Ferrite, Inductor_SMD:L_0805_2012Metric, F.Cu at (40.8, 177.2)
- added L17: L_Ferrite, Inductor_SMD:L_0805_2012Metric, F.Cu at (40.8, 179.9)
- added L18: L_Ferrite, Inductor_SMD:L_0805_2012Metric, F.Cu at (40.8, 182.7)
- added L19: L_Ferrite, Inductor_SMD:L_0805_2012Metric, F.Cu at (70.4, 112.3)
- added L2: 8.2uH, Inductor_SMD:L_Sunlord_MWSA0603S, F.Cu at (36.5, 105.5)
- added L20: L_Ferrite, Inductor_SMD:L_0805_2012Metric, F.Cu at (70.4, 115.0)
- added L21: L_Ferrite, Inductor_SMD:L_0805_2012Metric, F.Cu at (70.4, 117.8)
- added L22: L_Ferrite, Inductor_SMD:L_0805_2012Metric, F.Cu at (70.4, 120.5)
- added L23: L_Ferrite, Inductor_SMD:L_0805_2012Metric, F.Cu at (40.8, 143.4)
- added L24: L_Ferrite, Inductor_SMD:L_0805_2012Metric, F.Cu at (40.8, 146.1)
- added L25: L_Ferrite, Inductor_SMD:L_0805_2012Metric, F.Cu at (40.8, 148.9)
- added L26: L_Ferrite, Inductor_SMD:L_0805_2012Metric, F.Cu at (40.8, 151.6)
- added L3: L_Ferrite, Inductor_SMD:L_0805_2012Metric, F.Cu at (69.0, 143.4)
- added L4: L_Ferrite, Inductor_SMD:L_0805_2012Metric, F.Cu at (69.0, 146.1)
- added L5: L_Ferrite, Inductor_SMD:L_0805_2012Metric, F.Cu at (69.0, 148.9)
- added L6: L_Ferrite, Inductor_SMD:L_0805_2012Metric, F.Cu at (69.0, 151.6)
- added L7: L_Ferrite, Inductor_SMD:L_0805_2012Metric, F.Cu at (97.3, 143.4)
- added L8: L_Ferrite, Inductor_SMD:L_0805_2012Metric, F.Cu at (97.3, 146.1)
- added L9: L_Ferrite, Inductor_SMD:L_0805_2012Metric, F.Cu at (97.3, 148.9)
- added Q1: WSF3087, Package_TO_SOT_SMD:SOT-23, F.Cu at (83.5, 188.3)
- added Q2: WSF3087, Package_TO_SOT_SMD:SOT-23, F.Cu at (65.5, 188.3)
- added Q3: WSF3087, Package_TO_SOT_SMD:SOT-23, F.Cu at (47.6, 188.3)
- added Q4: WSF3087, Package_TO_SOT_SMD:SOT-23, F.Cu at (47.6, 172.2)
- added Q5: WSF3087, Package_TO_SOT_SMD:SOT-23, F.Cu at (83.5, 172.2)
- added Q6: WSF3087, Package_TO_SOT_SMD:SOT-23, F.Cu at (65.5, 172.2)
- added Q7: AO3400A, Package_TO_SOT_SMD:SOT-23, F.Cu at (219.7, 121.2)
- added Q8: AO3400A, Package_TO_SOT_SMD:SOT-23, F.Cu at (219.7, 125.8)
- added R1: 4.7k, Resistor_SMD:R_0805_2012Metric, F.Cu at (16.5, 102.8)
- added R10: 10k, Resistor_SMD:R_0805_2012Metric, F.Cu at (20.9, 114.7)
- added R11: 10k, Resistor_SMD:R_0805_2012Metric, F.Cu at (25.3, 102.8)
- added R12: 4.7k, Resistor_SMD:R_0805_2012Metric, F.Cu at (25.3, 105.8)
- added R13: 1k, Resistor_SMD:R_0805_2012Metric, F.Cu at (25.3, 108.8)
- added R14: 4.7kΩ, fab_R:R_0402, F.Cu at (58.4, 144.5)
- added R15: 4.7kΩ, fab_R:R_0402, F.Cu at (58.4, 149.4)
- added R16: 120m, Resistor_SMD:R_2512_6332Metric, F.Cu at (86.6, 144.5)
- added R17: 120m, Resistor_SMD:R_2512_6332Metric, F.Cu at (86.6, 149.4)
- added R18: 120m, Resistor_SMD:R_2512_6332Metric, F.Cu at (83.0, 118.9)
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Connections:
- C1 pad 1: Net-(U2-5VOUT) -> Net-(D2-A)
- C1 pad 2: GND -> Net-(D1-K)
- C10 pad 1: Net-(U5-5VOUT) -> GND
- C10 pad 2: GND -> +5V
- C11 pad 1: /A-driver/CPO -> +5V
- C11 pad 2: /A-driver/CPI -> GND
- C12 pad 1: Net-(U5-VCC) -> GND
- C12 pad 2: GND -> VDC
- C13 pad 1: Net-(U6-5VOUT) -> GND
- C13 pad 2: GND -> +5V (x2)
- C13 pad 1: Net-(U2-VCC) -> GND
- C14 pad 1: /B-driver/CPO -> GND
- C14 pad 2: /B-driver/CPI -> Net-(U3-COMP)
- C15 pad 1: Net-(U6-VCC) -> GND
- C15 pad 2: GND -> +5V
- C16 pad 1: Net-(U7-5VOUT) -> GND
- C16 pad 2: GND -> Net-(C16-Pad2)
- C17 pad 1: /C-driver/CPO -> +5V
- C17 pad 2: /C-driver/CPI -> GND
- C18 pad 1: Net-(U7-VCC) -> +3.3V
- C2 pad 1: /X-driver/CPO -> GND (x2)
- C2 pad 2: /X-driver/CPI -> Net-(C2-Pad2) (x2)
- C3 pad 1: Net-(U2-VCC) -> GND
- C3 pad 2: GND -> Net-(C2-Pad2)
- C4 pad 1: Net-(U3-5VOUT) -> GND
- C4 pad 2: GND -> VDC
- C5 pad 1: /Y-driver/CPO -> GND
- C5 pad 2: /Y-driver/CPI -> VDC
- C6 pad 1: Net-(U3-VCC) -> VDC
- C7 pad 1: Net-(U4-5VOUT) -> GND
- C7 pad 2: GND -> /PSU/VIN (x2)
- C7 pad 1: Net-(U2-5VOUT) -> GND
- C8 pad 1: /Z-driver/CPO -> Net-(D4-K)
- C8 pad 2: /Z-driver/CPI -> Net-(U3-BOOT)
- C9 pad 1: Net-(U4-VCC) -> GND
- C9 pad 2: GND -> VDC
- U1 pad 1: +3.3V -> Net-(D1-K)
- U1 pad 2: unconnected-(U1-LNA_IN-Pad2) -> Net-(D1-K)
- U1 pad 3: +3.3V -> Net-(D1-K)
- U1 pad 4: +3.3V -> Net-(D1-A)
- U1 pad 5: /CPU/VAC_PUMP -> /PSU/VIN
- U1 pad 6: /CPU/AIR1 -> /PSU/VIN
- U1 pad 7: /CPU/AIR2 -> /PSU/VIN
- U1 pad 8: /CPU/AIR_PUMP -> /PSU/VIN
- U2 pad 1: unconnected-(U2-TST_MODE-Pad1) -> Net-(D1-K)
- U2 pad 2: unconnected-(U2-CLK-Pad2) -> Net-(D1-K)
- U2 pad 3: /CPU/SPI_CS_X -> Net-(D1-K)
- U2 pad 4: /A-driver/SPI_CLK -> Net-(D2-A)
- U2 pad 5: /A-driver/SPI_MOSI -> Net-(C2-Pad2)
- U2 pad 6: unconnected-(U2-NC-Pad6) -> Net-(C2-Pad2)
- U2 pad 7: /A-driver/SPI_MISO -> Net-(C2-Pad2)
- U2 pad 8: unconnected-(U2-REFL_STEP-Pad8) -> Net-(C2-Pad2)
- U3 pad 1: unconnected-(U3-TST_MODE-Pad1) -> Net-(U3-BOOT)
- U3 pad 2: unconnected-(U3-CLK-Pad2) -> VDC
- U3 pad 3: /CPU/SPI_CS_Y -> Net-(U3-EN)
- U3 pad 4: /A-driver/SPI_CLK -> Net-(U3-RT/CLK)
- U3 pad 5: /A-driver/SPI_MOSI -> Net-(U3-FB)
- U3 pad 6: unconnected-(U3-NC-Pad6) -> Net-(U3-COMP)
- U3 pad 7: /A-driver/SPI_MISO -> GND
- U3 pad 8: unconnected-(U3-REFL_STEP-Pad8) -> Net-(D4-K)
- U3 pad 9: unconnected-(U3-REFR_DIR-Pad9) -> GND
- U4 pad 1: unconnected-(U4-TST_MODE-Pad1) -> GND
- U4 pad 2: unconnected-(U4-CLK-Pad2) -> +3.3V
- U4 pad 3: /CPU/SPI_CS_Z -> +5V
- U5 pad 2: unconnected-(U5-CLK-Pad2) -> +3.3V
- U5 pad 3: /A-driver/SPI_CS -> unconnected-(U5-NC-Pad3)
- U5 pad 4: /A-driver/SPI_CLK -> /CPU/I2C_SDA
- U5 pad 5: /A-driver/SPI_MOSI -> /CPU/I2C_SCL
- U5 pad 6: unconnected-(U5-NC-Pad6) -> GND
- U6 pad 1: unconnected-(U6-TST_MODE-Pad1) -> +3.3V
- U6 pad 10: unconnected-(U6-VCC_IO-Pad10) -> /CPU/VAC1
- U6 pad 11: unconnected-(U6-SD_MODE-Pad11) -> /CPU/VAC2
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Routing:
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
Commit message: update_PSU
Parts:
- removed C10, C15, C17, C18, C9: 10u, Capacitor_SMD:C_0805_2012Metric
- removed the C13 at (125.7, 106.9)
- removed the C13 at (137.7, 109.4)
- removed C16: 4.7n, Capacitor_SMD:C_0805_2012Metric
- removed C19, C20: 100n, Capacitor_SMD:C_0805_2012Metric
- removed the C2 at (82.3, 96.2)
- removed the C2 at (106.6, 85.4)
- removed the C7 at (125.7, 114.0)
- removed the C7 at (137.7, 106.9)
- removed D6, D7, D8: Green, LED_SMD:LED_0805_2012Metric
- removed F1: Fuse, Fuse:Fuseholder_Littelfuse_Nano2_154x
- removed L10, L11, L12, L13, L14, L15, L16, L17, L18, L19, L20, L21, L22, L23, L24, L25, L26, L4, L5, L6, L7, L8, L9: L_Ferrite, Inductor_SMD:L_0805_2012Metric
- removed L2: 8.2uH, Inductor_SMD:L_Sunlord_MWSA0603S
- removed Q8: AO3400A, Package_TO_SOT_SMD:SOT-23
- removed R11, R5: 10k, Resistor_SMD:R_0805_2012Metric
- removed R12: 4.7k, Resistor_SMD:R_0805_2012Metric
- removed R13, R71: 1k, Resistor_SMD:R_0805_2012Metric
- removed R6: 53.6k, Resistor_SMD:R_0805_2012Metric
- removed R7: 16.9k, Resistor_SMD:R_0805_2012Metric
- removed TP4: TestPoint, TestPoint:TestPoint_Pad_D2.0mm
- removed U1: FDS4435BZ, Package_SO:SO-8_3.9x4.9mm_P1.27mm
- removed U24: PESD5V2S2UT, Package_TO_SOT_SMD:SOT-23-3
- removed U25, U26, U27: PESD3V3S2UT, Package_TO_SOT_SMD:SOT-23-3
- added C105: 4.7uF, fab_C:C_0603, F.Cu at (120.5, 38.1)
- added C106: 470pF, fab_C:C_0805, F.Cu at (128.8, 58.1)
- added C107: 470pF, fab_C:C_0805, F.Cu at (128.8, 61.0)
- added C108: 470pF, fab_C:C_0805, F.Cu at (128.8, 64.0)
- added C109: 22nF, fab_C:C_0603, F.Cu at (120.5, 40.6)
- added C110: 470pF, fab_C:C_0805, F.Cu at (133.2, 58.1)
- added C111: 470pF, fab_C:C_0805, F.Cu at (133.2, 61.0)
- added C112: 100nF, fab_C:C_0603, F.Cu at (120.5, 43.2)
- added C113: 100nF, fab_C:C_0603, F.Cu at (120.5, 45.7)
- added C114: 100uF/50V, fab_C_Pol:CP_Elec_8x10.5, F.Cu at (133.3, 51.6)
- added C115: 10uF, fab_C:C_1210, F.Cu at (143.9, 39.0)
- added C116: 100nF, fab_C:C_0603, F.Cu at (120.5, 48.2)
- added C117: 100nF, fab_C:C_0603, F.Cu at (120.5, 50.7)
- added C118: 100nF, fab_C:C_0603, F.Cu at (120.5, 53.2)
- added C13: 100nF, fab_C:C_0603, F.Cu at (42.8, 66.2)
- added C2: 10uF, fab_C:C_1210, F.Cu at (43.6, 39.0)
- added C7: 100uF/50V, fab_C_Pol:CP_Elec_8x10.5, F.Cu at (68.5, 41.9)
- added D22: LESD5D5.0CT1G, fab_D:SOD-523, F.Cu at (137.4, 146.5)
- added D23: LESD5D5.0CT1G, fab_D:SOD-523, F.Cu at (155.3, 113.9)
- added D24: GREEN, fab_D:LED_0603_1608Metric, F.Cu at (79.0, 69.3)
- added D25: GREEN, fab_D:LED_0603_1608Metric, F.Cu at (79.0, 71.9)
- added F2: 01550900M, fab_F:Fuseholder_Littelfuse_Nano2_154x, F.Cu at (46.8, 78.2)
- added FB1: FerriteBead, fab_R:R_0805, F.Cu at (117.0, 62.0)
- added FB10: FerriteBead, fab_R:R_0805, F.Cu at (59.9, 137.8)
- added FB11: FerriteBead, fab_R:R_0805, F.Cu at (59.9, 140.7)
- added FB12: FerriteBead, fab_R:R_0805, F.Cu at (59.9, 143.7)
- added FB13: FerriteBead, fab_R:R_0805, F.Cu at (133.2, 97.0)
- added FB14: FerriteBead, fab_R:R_0805, F.Cu at (137.6, 91.2)
- added FB15: FerriteBead, fab_R:R_0805, F.Cu at (137.6, 94.1)
- added FB16: FerriteBead, fab_R:R_0805, F.Cu at (137.6, 97.0)
- added FB17: FerriteBead, fab_R:R_0805, F.Cu at (55.5, 110.6)
- added FB18: FerriteBead, fab_R:R_0805, F.Cu at (59.9, 104.7)
- added FB19: FerriteBead, fab_R:R_0805, F.Cu at (59.9, 107.7)
- added FB2: FerriteBead, fab_R:R_0805, F.Cu at (103.0, 58.1)
- added FB20: FerriteBead, fab_R:R_0805, F.Cu at (59.9, 110.6)
- added FB21: FerriteBead, fab_R:R_0805, F.Cu at (133.2, 64.0)
- added FB22: FerriteBead, fab_R:R_0805, F.Cu at (137.6, 58.1)
- added FB23: FerriteBead, fab_R:R_0805, F.Cu at (137.6, 61.0)
- added FB24: FerriteBead, fab_R:R_0805, F.Cu at (137.6, 64.0)
- added FB3: FerriteBead, fab_R:R_0805, F.Cu at (103.0, 61.0)
- added FB4: FerriteBead, fab_R:R_0805, F.Cu at (103.0, 64.0)
- added FB5: FerriteBead, fab_R:R_0805, F.Cu at (98.6, 97.0)
- added FB6: FerriteBead, fab_R:R_0805, F.Cu at (103.0, 91.2)
- added FB7: FerriteBead, fab_R:R_0805, F.Cu at (103.0, 94.1)
- added FB8: FerriteBead, fab_R:R_0805, F.Cu at (103.0, 97.0)
- added FB9: FerriteBead, fab_R:R_0805, F.Cu at (55.5, 143.7)
- added R50: 10kΩ, fab_R:R_0402, F.Cu at (134.2, 146.3)
- added R51: 1kΩ, fab_R:R_0402, F.Cu at (134.2, 148.2)
- added R52: 10kΩ, fab_R:R_0402, F.Cu at (152.1, 113.7)
- added R54: 442kΩ, fab_R:R_0603, F.Cu at (54.8, 68.7)
- added R55: 90.9kΩ, fab_R:R_0603, F.Cu at (54.8, 71.2)
- added R56: 10.2kΩ, fab_R:R_0603, F.Cu at (54.8, 73.7)
- added TP38: TestPoint, TestPoint:TestPoint_Pad_D2.0mm, F.Cu at (59.8, 55.1)
- C1, C102, C103, C104, C42, C43, C46, C47, C48, C56, C57, C60, C61, C62, C70, C71, C74, C75, C76, C84, C85, C88, C89, C90, C98, C99: value 100n -> 100nF; footprint Capacitor_SMD:C_0805_2012Metric -> fab_C:C_0603
- C100, C44, C58, C72, C86: value 100u -> 100uF/50V; footprint Capacitor_SMD:CP_Elec_6.3x7.7 -> fab_C_Pol:CP_Elec_8x10.5
- C101, C12, C3, C4, C45, C5, C59, C73, C87: value 10u -> 10uF; footprint Capacitor_SMD:C_0805_2012Metric -> fab_C:C_1210
- C11, C6: value 100u -> 10uF; footprint Capacitor_SMD:CP_Elec_6.3x7.7 -> fab_C:C_1210
- C14: value 47p -> 100nF; footprint Capacitor_SMD:C_0805_2012Metric -> fab_C:C_0603
- C21: value 4.7uF -> 100nF
- C22: value 470nF -> 10uF; footprint fab_C:C_0603 -> fab_C:C_1210
- C23, C25: value 470p -> 10uF; footprint Capacitor_SMD:C_0805_2012Metric -> fab_C:C_1210
- C24: value 22nF/0805 -> 10uF; footprint fab_C:C_0805 -> fab_C:C_1210
- C26: value 470p -> 100nF; footprint Capacitor_SMD:C_0805_2012Metric -> fab_C:C_0603
- C27: value 470p -> 22uF; footprint Capacitor_SMD:C_0805_2012Metric -> fab_C:C_1210
- C28, C29: value 100n -> 22uF; footprint Capacitor_SMD:C_0805_2012Metric -> fab_C:C_1210
- C30: value 100u -> 22uF; footprint Capacitor_SMD:CP_Elec_6.3x7.7 -> fab_C:C_1210
- C31: value 10u -> 47pF; footprint Capacitor_SMD:C_0805_2012Metric -> fab_C:C_0603
- C32: value 100n -> 4.7nF; footprint Capacitor_SMD:C_0805_2012Metric -> fab_C:C_0603
- C36, C50, C64, C78, C92: value 470nF -> 470pF; footprint fab_C:C_0603 -> fab_C:C_0805
- C37, C40, C41, C51, C54, C55, C65, C68, C69, C79, C82, C83, C93, C96, C97: value 470p -> 470pF; footprint Capacitor_SMD:C_0805_2012Metric -> fab_C:C_0805
- C38, C52, C66, C80, C94: value 22nF/0805 -> 470pF
- C39, C53, C67, C81, C95: value 470p -> 22nF; footprint Capacitor_SMD:C_0805_2012Metric -> fab_C:C_0603
- C8: value 100n -> 100uF/50V; footprint Capacitor_SMD:C_0805_2012Metric -> fab_C_Pol:CP_Elec_8x10.5
- D1, D2: value BZT52C16 -> SQJ479EP-T1_GE3; footprint Diode_SMD:D_SOD-123 -> fab_T:PowerPAK_SO-8L_Single
- D10: value SM4007 -> B560C; footprint Diode_SMD:D_SOD-123F -> fab_D:SMC
- D17, D18: value LESD5D5.0CT1G -> SM4007; footprint fab_D:SOD-523 -> Diode_SMD:D_SOD-123F
- D3: value SMF28A -> BZT52C16; footprint Diode_SMD:D_SMF -> fab_D:SOD-123
- D4: value B560C -> BZT52C16; footprint Diode_SMD:D_SMC -> fab_D:SOD-123
- D5: value SS34 -> SMF28A; footprint Diode_SMD:D_SMA -> fab_D:SOD-123FL
- D9: value SM4007 -> GREEN; footprint Diode_SMD:D_SOD-123F -> fab_D:LED_0603_1608Metric
- J10, J11, J12, J13, J9: value FET -> Conn_01x02_Pin; footprint Connector_JST:JST_PH_B2B-PH-SM4-TB_1x02-1MP_P2.00mm_Vertical -> fab_CON:WE_620302124022
- J14: value TOP_LIGHT -> Conn_01x02_Pin; footprint Connector_JST:JST_PH_B3B-PH-SM4-TB_1x03-1MP_P2.00mm_Vertical -> fab_CON:WE_620302124022
- J15, J17, J18, J19, J20, J21: value TOP_LIGHT -> Conn_01x03_Pin; footprint Connector_JST:JST_PH_B3B-PH-SM4-TB_1x03-1MP_P2.00mm_Vertical -> fab_CON:WE_620303124022
- J16: value FAN -> Conn_01x03_Pin; footprint Connector_JST:JST_PH_B2B-PH-SM4-TB_1x02-1MP_P2.00mm_Vertical -> fab_CON:WE_620303124022
- J2: value MOTOR -> FAN; footprint Connector_JST:JST_PH_B4B-PH-SM4-TB_1x04-1MP_P2.00mm_Vertical -> Connector_JST:JST_PH_B2B-PH-SM4-TB_1x02-1MP_P2.00mm_Vertical
- J3, J4, J5, J6, J7: value MOTOR -> Conn_01x04_Pin; footprint Connector_JST:JST_PH_B4B-PH-SM4-TB_1x04-1MP_P2.00mm_Vertical -> fab_CON:WE_620304124022
- J8: value FET -> Conn_01x04_Pin; footprint Connector_JST:JST_PH_B2B-PH-SM4-TB_1x02-1MP_P2.00mm_Vertical -> fab_CON:WE_620304124022
- L1: value 2.2u -> 2.2uH; footprint Inductor_SMD:L_Sunlord_MWSA0402S -> fab_L:L_Sunlord_MWSA0402S
- L3: value L_Ferrite -> 8.2uH; footprint Inductor_SMD:L_0805_2012Metric -> fab_L:L_Changjiang_FXL0630
- Q1, Q2, Q3, Q4, Q5, Q6: value WSF3087 -> AO3400A
- R1, R2: value 4.7k -> 4.7kΩ; footprint Resistor_SMD:R_0805_2012Metric -> fab_R:R_0603
- R10, R3, R4: value 10k -> 10kΩ; footprint Resistor_SMD:R_0805_2012Metric -> fab_R:R_0603
- R14: value 4.7kΩ -> 53.6kΩ; footprint fab_R:R_0402 -> fab_R:R_0603
- R15: value 4.7kΩ -> 16.9kΩ; footprint fab_R:R_0402 -> fab_R:R_0603
- R16: value 120m -> 243kΩ; footprint Resistor_SMD:R_2512_6332Metric -> fab_R:R_0603
- R17, R18: value 120m -> 4.7kΩ; footprint Resistor_SMD:R_2512_6332Metric -> fab_R:R_0402
- R19: value 120m -> 1k; footprint Resistor_SMD:R_2512_6332Metric -> Resistor_SMD:R_0805_2012Metric
- R20, R21, R22, R23, R24, R25, R26, R27: value 120m -> 120mΩ; footprint Resistor_SMD:R_2512_6332Metric -> fab_R:R_2512
- R28, R30: value 1k -> 120mΩ; footprint Resistor_SMD:R_0805_2012Metric -> fab_R:R_2512
- R29, R31: value 10k -> 120mΩ; footprint Resistor_SMD:R_0805_2012Metric -> fab_R:R_2512
- R40, R42: value 10kΩ -> 1k; footprint fab_R:R_0402 -> Resistor_SMD:R_0805_2012Metric
- R41, R43: value 10kΩ -> 10k; footprint fab_R:R_0402 -> Resistor_SMD:R_0805_2012Metric
- R46, R48: value 1kΩ -> 10kΩ
- R53: value 1k -> 1kΩ; footprint Resistor_SMD:R_0805_2012Metric -> fab_R:R_0402
- R8: value 4.7k -> 1kΩ; footprint Resistor_SMD:R_0805_2012Metric -> fab_R:R_0603
- R9: value 243k -> 4.7kΩ; footprint Resistor_SMD:R_0805_2012Metric -> fab_R:R_0603
- U2: value FDS4435BZ -> AMS1117-3.3; footprint Package_SO:SO-8_3.9x4.9mm_P1.27mm -> fab_U:SOT-223
- U3: value TPS54560BDDA -> TPS54560BDDAR; footprint Package_SO:Texas_R-PDSO-G8_EP2.95x4.9mm_Mask2.4x3.1mm_ThermalVias -> fab_U:Texas_HSOP-8-1EP_3.9x4.9mm_P1.27mm_ThermalVias
- U4: value AP1117-33 -> XGZP6857D; footprint Package_TO_SOT_SMD:SOT-223-3_TabPin2 -> Package_DIP:DIP-6_W10.16mm
- U5: value XGZP6857D -> ESP32-PICO-V3; footprint Package_DIP:DIP-6_W10.16mm -> Package_DFN_QFN:QFN-48-1EP_7x7mm_P0.5mm_EP5.15x5.15mm
- U6: value ESP32-PICO-V3 -> XGZP6857D; footprint Package_DFN_QFN:QFN-48-1EP_7x7mm_P0.5mm_EP5.15x5.15mm -> Package_DIP:DIP-6_W10.16mm
- U7: value XGZP6857D -> FE1.1S-BQFN24B; footprint Package_DIP:DIP-6_W10.16mm -> fab_U:WQFN-24-1EP_4x4mm_P0.5mm_EP2.7x2.7mm
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Connections:
- C1 pad 1: Net-(D2-A) -> Net-(D1-S)
- C1 pad 2: Net-(D1-K) -> Net-(D2-G)
- C101 pad 1: GND -> VDC
- C101 pad 2: VDC -> GND
- C102 pad 1: GND -> unconnected-(C102-Pad1)
- C102 pad 2: VDC -> GND
- C103 pad 1: GND -> unconnected-(C103-Pad1)
- C103 pad 2: VDC -> GND
- C104 pad 1: GND -> +3.3V
- C104 pad 2: +3.3V -> GND
- C11 pad 1: +5V -> +3.3V
- C12 pad 1: GND -> +5V
- C12 pad 2: VDC -> GND
- C14 pad 1: GND -> +5V
- C14 pad 2: Net-(U3-COMP) -> GND
- C21 pad 1: Net-(U8-5VOUT) -> Net-(U3-BOOT)
- C21 pad 2: GND -> Net-(D10-A1)
- C22 pad 1: Net-(U8-VCC) -> VDC
- C23 pad 1: GND -> VDC
- C23 pad 2: /X-driver/A1 -> GND
- C24 pad 1: /X-driver/CPO -> VDC
- C24 pad 2: /X-driver/CPI -> GND
- C25 pad 1: /X-driver/A2 -> VDC
- C26 pad 1: GND -> VDC
- C26 pad 2: /X-driver/B1 -> GND
- C27 pad 1: /X-driver/B2 -> +5V
- C28 pad 1: GND -> +5V
- C28 pad 2: Net-(U8-BRB) -> GND
- C29 pad 1: GND -> +5V
- C29 pad 2: Net-(U8-BRA) -> GND
- C3 pad 1: GND -> Net-(D2-D)
- C3 pad 2: Net-(C2-Pad2) -> GND
- C30 pad 1: VDC -> +5V
- C31 pad 1: GND -> Net-(U3-COMP)
- C31 pad 2: VDC -> GND
- C32 pad 1: GND -> Net-(C32-Pad1)
- C32 pad 2: VDC -> GND
- C33 pad 1: GND -> +3.3V
- C33 pad 2: VDC -> GND
- C34 pad 1: GND -> +3.3V
- C34 pad 2: +3.3V -> GND
- C35 pad 1: Net-(U9-5VOUT) -> Net-(U8-5VOUT)
- C36 pad 1: Net-(U9-VCC) -> Net-(U8-VCC)
- C37 pad 1: GND -> /X-driver/A1
- C37 pad 2: /Y-driver/A1 -> GND
- C38 pad 1: /Y-driver/CPO -> GND
- C38 pad 2: /Y-driver/CPI -> /X-driver/A2
- C39 pad 1: /Y-driver/A2 -> /X-driver/CPO
- C39 pad 2: GND -> /X-driver/CPI
- C4 pad 1: GND -> Net-(D2-D)
- C4 pad 2: VDC -> GND
- C40 pad 1: GND -> /X-driver/B1
- C40 pad 2: /Y-driver/B1 -> GND
- C41 pad 1: /Y-driver/B2 -> GND
- C41 pad 2: GND -> /X-driver/B2
- C42 pad 1: GND -> Net-(U8-BRB)
- C42 pad 2: Net-(U9-BRB) -> GND
- C43 pad 1: GND -> Net-(U8-BRA)
- C43 pad 2: Net-(U9-BRA) -> GND
- C45 pad 1: GND -> VDC
- C45 pad 2: VDC -> GND
- C46 pad 1: GND -> unconnected-(C46-Pad1)
- C46 pad 2: VDC -> GND
- C47 pad 1: GND -> unconnected-(C47-Pad1)
- C47 pad 2: VDC -> GND
- C48 pad 1: GND -> +3.3V
- C48 pad 2: +3.3V -> GND
- C49 pad 1: Net-(U10-5VOUT) -> Net-(U9-5VOUT)
- C5 pad 1: GND -> VDC
- C5 pad 2: VDC -> GND
- C50 pad 1: Net-(U10-VCC) -> Net-(U9-VCC)
- C51 pad 1: GND -> /Y-driver/A1
- C51 pad 2: /Z-driver/A1 -> GND
- C52 pad 1: /Z-driver/CPO -> GND
- C52 pad 2: /Z-driver/CPI -> /Y-driver/A2
- C53 pad 1: /Z-driver/A2 -> /Y-driver/CPO
- C53 pad 2: GND -> /Y-driver/CPI
- C54 pad 1: GND -> /Y-driver/B1
- C54 pad 2: /Z-driver/B1 -> GND
- C55 pad 1: /Z-driver/B2 -> GND
- C55 pad 2: GND -> /Y-driver/B2
- C56 pad 1: GND -> Net-(U9-BRB)
- C56 pad 2: Net-(U10-BRB) -> GND
- C57 pad 1: GND -> Net-(U9-BRA)
- C57 pad 2: Net-(U10-BRA) -> GND
- C59 pad 1: GND -> VDC
- C59 pad 2: VDC -> GND
- C60 pad 1: GND -> unconnected-(C60-Pad1)
- C60 pad 2: VDC -> GND
- C61 pad 1: GND -> unconnected-(C61-Pad1)
- C61 pad 2: VDC -> GND
- C62 pad 1: GND -> +3.3V
- C62 pad 2: +3.3V -> GND
- C63 pad 1: Net-(U11-5VOUT) -> Net-(U10-5VOUT)
- C64 pad 1: Net-(U11-VCC) -> Net-(U10-VCC)
- C65 pad 1: GND -> /Z-driver/A1
- C65 pad 2: /A-driver/A1 -> GND
- C66 pad 1: /A-driver/CPO -> GND
- C66 pad 2: /A-driver/CPI -> /Z-driver/A2
- C67 pad 1: /A-driver/A2 -> /Z-driver/CPO
- C67 pad 2: GND -> /Z-driver/CPI
- C68 pad 1: GND -> /Z-driver/B1
- C68 pad 2: /A-driver/B1 -> GND
- C69 pad 1: /A-driver/B2 -> GND
- C69 pad 2: GND -> /Z-driver/B2
- C70 pad 1: GND -> Net-(U10-BRB)
- C70 pad 2: Net-(U11-BRB) -> GND
- C71 pad 1: GND -> Net-(U10-BRA)
- C71 pad 2: Net-(U11-BRA) -> GND
- C73 pad 1: GND -> VDC
- C73 pad 2: VDC -> GND
- C74 pad 1: GND -> unconnected-(C74-Pad1)
- C74 pad 2: VDC -> GND
- C75 pad 1: GND -> unconnected-(C75-Pad1)
- C75 pad 2: VDC -> GND
- C76 pad 1: GND -> +3.3V
- C76 pad 2: +3.3V -> GND
- C77 pad 1: Net-(U12-5VOUT) -> Net-(U11-5VOUT)
- C78 pad 1: Net-(U12-VCC) -> Net-(U11-VCC)
- C79 pad 1: GND -> /A-driver/A1
- C79 pad 2: /B-driver/A1 -> GND
- C8 pad 1: Net-(D4-K) -> VDC
- C8 pad 2: Net-(U3-BOOT) -> GND
- C80 pad 1: /B-driver/CPO -> GND
- C80 pad 2: /B-driver/CPI -> /A-driver/A2
- C81 pad 1: /B-driver/A2 -> /A-driver/CPO
- C81 pad 2: GND -> /A-driver/CPI
- C82 pad 1: GND -> /A-driver/B1
- C82 pad 2: /B-driver/B1 -> GND
- C83 pad 1: /B-driver/B2 -> GND
- C83 pad 2: GND -> /A-driver/B2
- C84 pad 1: GND -> Net-(U11-BRB)
- C84 pad 2: Net-(U12-BRB) -> GND
- C85 pad 1: GND -> Net-(U11-BRA)
- C85 pad 2: Net-(U12-BRA) -> GND
- C87 pad 1: GND -> VDC
- C87 pad 2: VDC -> GND
- C88 pad 1: GND -> unconnected-(C88-Pad1)
- C88 pad 2: VDC -> GND
- C89 pad 1: GND -> unconnected-(C89-Pad1)
- C89 pad 2: VDC -> GND
- C90 pad 1: GND -> +3.3V
- C90 pad 2: +3.3V -> GND
- C91 pad 1: Net-(U13-5VOUT) -> Net-(U12-5VOUT)
- C92 pad 1: Net-(U13-VCC) -> Net-(U12-VCC)
- C93 pad 1: GND -> /B-driver/A1
- C93 pad 2: /C-driver/A1 -> GND
- C94 pad 1: /C-driver/CPO -> GND
- C94 pad 2: /C-driver/CPI -> /B-driver/A2
- C95 pad 1: /C-driver/A2 -> /B-driver/CPO
- C95 pad 2: GND -> /B-driver/CPI
- C96 pad 1: GND -> /B-driver/B1
- C96 pad 2: /C-driver/B1 -> GND
- C97 pad 1: /C-driver/B2 -> GND
- C97 pad 2: GND -> /B-driver/B2
- C98 pad 1: GND -> Net-(U12-BRB)
- C98 pad 2: Net-(U13-BRB) -> GND
- C99 pad 1: GND -> Net-(U12-BRA)
- C99 pad 2: Net-(U13-BRA) -> GND
- D1 pad 1: Net-(D1-K) -> Net-(D1-S)
- D1 pad 2: Net-(D1-A) -> Net-(D1-G)
- D10 pad 1: VDC -> Net-(D10-A1)
- D10 pad 2: Net-(D10-A) -> GND
- D11 pad 1: VDC -> +5V
- D11 pad 2: Net-(D11-A) -> Net-(BZ1-+)
- D12 pad 1: VDC -> +5V
- D12 pad 2: Net-(D12-A) -> GND
- D15 pad 1: +5V -> VDC
- D15 pad 2: Net-(BZ1-+) -> Net-(D15-A)
- D16 pad 1: +5V -> VDC
- D17 pad 1: GND -> VDC
- D17 pad 2: Net-(D17-A2) -> Net-(D17-A)
- D18 pad 1: GND -> VDC
- D18 pad 2: Net-(D18-A2) -> Net-(D18-A)
- D2 pad 1: Net-(D1-K) -> Net-(D1-S)
- D2 pad 2: Net-(D2-A) -> Net-(D2-G)
- D3 pad 1: /PSU/VIN -> Net-(D1-S)
- D3 pad 2: GND -> Net-(D1-G)
- D4 pad 1: Net-(D4-K) -> Net-(D1-S)
- D4 pad 2: GND -> Net-(D2-G)
- D5 pad 1: +5V -> /PSU/VIN
- D5 pad 2: VBUS -> GND
- D9 pad 1: VDC -> GND
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Routing:
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Other:
- board outline removed
- board text removed: "https://github.com/palo-krnac/pnp32"
- board text removed: "pnp32"
