File: HARDWARE/pnp32_controller/pnp32_mainboard/wled.kicad_sch (KiCad schematic)
At the start: 4 parts, among them J14 TOP_LIGHT, U20 SN74LVC2G34, U21 PESD5V2S2UT

Commit message: update_PSU
Parts:
- removed J14: TOP_LIGHT, Connector_JST:JST_PH_B3B-PH-SM4-TB_1x03-1MP_P2.00mm_Vertical, symbol Connector_Generic_MountingPin:Conn_01x03_MountingPin
- added J15: Conn_01x03_Pin, fab_CON:WE_620303124022, symbol fab_CON:WE_620303124022
Connections:
- net +5V: now also J15.1 (Pin_1)
- net GND: now also J15.3 (Pin_3)
- net at TP36.1, U20.6 (1Y), U21.1: now also J15.2 (Pin_2)
Changed lines of the file:
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@@
-	(wire
-		(pts
-			(xy 204.47 97.79) (xy 204.47 92.71)
-		)
-		(stroke
-			(width 0)
-			(type default)
-		)
-	)
 	(wire
 		(pts
@@
 	)
 	(symbol
-		(lib_id "power:GND")
-		(at 204.47 97.79 0)
-		(unit 1)
-		(exclude_from_sim no)
-		(in_bom yes)
-		(on_board yes)
-		(dnp no)
-		(property "Reference" "#PWR0141"
-			(at 204.47 104.14 0)
-			(effects
-				(font
-					(size 1 1)
-				)
-				(hide yes)
-			)
-		)
-		(property "Value" "GND"
-			(at 204.47 100.33 90)
-			(effects
-				(font
-					(size 1 1)
-				)
-				(justify right)
-			)
-		)
-		(property "Footprint" ""
-			(at 204.47 97.79 0)
-			(effects
-				(font
-					(size 1 1)
-					(color 223 129 255 1)
-				)
-				(hide yes)
-			)
-		)
-		(property "Datasheet" ""
-			(at 204.47 97.79 0)
-			(effects
-				(font
-					(size 1 1)
-					(color 223 129 255 1)
-				)
-				(hide yes)
-			)
-		)
-		(property "Description" ""
-			(at 204.47 97.79 0)
-			(effects
-				(font
-					(size 1.27 1.27)
-				)
-				(hide yes)
-			)
-		)
-		(pin "1"
-		)
-		(instances
-			(project "pnp32_mainboard"
-				(path "/a02e5dd1-80da-4253-b87a-c8707aa3e0b0/68017b66-d25d-4af8-bffb-a371ea1e6e65"
-					(reference "#PWR0148")
-					(unit 1)
-				)
-				(path "/a02e5dd1-80da-4253-b87a-c8707aa3e0b0/d75b9ede-8115-4a1a-ba5c-5202cedca149"
-					(reference "#PWR0141")
-					(unit 1)
-				)
-			)
-		)
-	)
-	(symbol
-		(lib_id "Connector_Generic_MountingPin:Conn_01x03_MountingPin")
-		(at 204.47 85.09 0)
-		(unit 1)
-		(exclude_from_sim no)
-		(in_bom yes)
-		(on_board yes)
-		(dnp no)
-		(property "Reference" "J14"
-			(at 204.47 75.692 0)
-			(effects
-				(font
-					(size 1.27 1.27)
-				)
-			)
-		)
-		(property "Value" "TOP_LIGHT"
-			(at 204.47 78.74 0)
-			(effects
-				(font
-					(size 1.27 1.27)
-				)
-			)
-		)
-		(property "Footprint" "Connector_JST:JST_PH_B3B-PH-SM4-TB_1x03-1MP_P2.00mm_Vertical"
-			(at 204.47 85.09 0)
-			(effects
-				(font
-					(size 1.27 1.27)
-				)
-				(hide yes)
-			)
-		)
-		(property "Datasheet" "~"
-			(at 204.47 85.09 0)
-			(effects
-				(font
-					(size 1.27 1.27)
-				)
-				(hide yes)
-			)
-		)
-		(property "Description" ""
-			(at 204.47 85.09 0)
-			(effects
-				(font
-					(size 1.27 1.27)
-				)
-				(hide yes)
-			)
-		)
-		(property "JLCPCB" "C146054"
-			(at 204.47 85.09 0)
-			(effects
-				(font
-					(size 1.27 1.27)
-				)
-				(hide yes)
-			)
-		)
-		(property "LCSC" "C2829151"
-			(at 204.47 85.09 0)
-			(effects
-				(font
-					(size 1.27 1.27)
-				)
-				(hide yes)
-			)
-		)
-		(pin "3"
-		)
-		(pin "MP"
-		)
-		(pin "1"
-		)
-		(pin "2"
-		)
-		(instances
-			(project "pnp32_mainboard"
-				(path "/a02e5dd1-80da-4253-b87a-c8707aa3e0b0/68017b66-d25d-4af8-bffb-a371ea1e6e65"
-					(reference "J14")
-					(unit 1)
-				)
-				(path "/a02e5dd1-80da-4253-b87a-c8707aa3e0b0/d75b9ede-8115-4a1a-ba5c-5202cedca149"
-					(reference "J14")
-					(unit 1)
-				)
-			)
-		)
-	)
-	(symbol
 		(lib_id "index:SN74LVC2G34")
 		(at 151.765 100.33 0)
@@
 		(dnp no)
 		(fields_autoplaced yes)
-		(property "Reference" "#PWR0147"
+		(property "Reference" "#PWR0158"
 			(at 179.07 126.365 0)
 			(effects
@@
 			(project "pnp32_mainboard"
 				(path "/a02e5dd1-80da-4253-b87a-c8707aa3e0b0/68017b66-d25d-4af8-bffb-a371ea1e6e65"
-					(reference "#PWR0154")
-					(unit 1)
-				)
-				(path "/a02e5dd1-80da-4253-b87a-c8707aa3e0b0/d75b9ede-8115-4a1a-ba5c-5202cedca149"
-					(reference "#PWR0147")
+					(reference "#PWR0163")
+					(unit 1)
+				)
+				(path "/a02e5dd1-80da-4253-b87a-c8707aa3e0b0/d75b9ede-8115-4a1a-ba5c-5202cedca149"
+					(reference "#PWR0158")
 					(unit 1)
 				)
@@
 		(dnp no)
 		(fields_autoplaced yes)
-		(property "Reference" "#PWR0145"
+		(property "Reference" "#PWR0156"
 			(at 135.255 95.25 0)
 			(effects
@@
 			(project "pnp32_mainboard"
 				(path "/a02e5dd1-80da-4253-b87a-c8707aa3e0b0/68017b66-d25d-4af8-bffb-a371ea1e6e65"
-					(reference "#PWR0152")
-					(unit 1)
-				)
-				(path "/a02e5dd1-80da-4253-b87a-c8707aa3e0b0/d75b9ede-8115-4a1a-ba5c-5202cedca149"
-					(reference "#PWR0145")
+					(reference "#PWR0161")
+					(unit 1)
+				)
+				(path "/a02e5dd1-80da-4253-b87a-c8707aa3e0b0/d75b9ede-8115-4a1a-ba5c-5202cedca149"
+					(reference "#PWR0156")
 					(unit 1)
 				)
@@
 		(dnp no)
 		(fields_autoplaced yes)
-		(property "Reference" "#PWR0146"
+		(property "Reference" "#PWR0157"
 			(at 157.48 95.25 0)
 			(effects
@@
 			(project "pnp32_mainboard"
 				(path "/a02e5dd1-80da-4253-b87a-c8707aa3e0b0/68017b66-d25d-4af8-bffb-a371ea1e6e65"
-					(reference "#PWR0153")
-					(unit 1)
-				)
-				(path "/a02e5dd1-80da-4253-b87a-c8707aa3e0b0/d75b9ede-8115-4a1a-ba5c-5202cedca149"
-					(reference "#PWR0146")
+					(reference "#PWR0162")
+					(unit 1)
+				)
+				(path "/a02e5dd1-80da-4253-b87a-c8707aa3e0b0/d75b9ede-8115-4a1a-ba5c-5202cedca149"
+					(reference "#PWR0157")
 					(unit 1)
 				)
@@
 		(dnp no)
 		(fields_autoplaced yes)
-		(property "Reference" "#PWR0143"
+		(property "Reference" "#PWR0154"
 			(at 196.85 78.74 0)
 			(effects
@@
 			(project "pnp32_mainboard"
 				(path "/a02e5dd1-80da-4253-b87a-c8707aa3e0b0/68017b66-d25d-4af8-bffb-a371ea1e6e65"
-					(reference "#PWR0143")
-					(unit 1)
-				)
-				(path "/a02e5dd1-80da-4253-b87a-c8707aa3e0b0/d75b9ede-8115-4a1a-ba5c-5202cedca149"
-					(reference "#PWR0143")
+					(reference "#PWR0159")
+					(unit 1)
+				)
+				(path "/a02e5dd1-80da-4253-b87a-c8707aa3e0b0/d75b9ede-8115-4a1a-ba5c-5202cedca149"
+					(reference "#PWR0154")
 					(unit 1)
 				)
@@
 		(on_board yes)
 		(dnp no)
-		(property "Reference" "#PWR0142"
+		(property "Reference" "#PWR0155"
 			(at 196.85 97.79 0)
 			(effects
@@
 			(project "pnp32_mainboard"
 				(path "/a02e5dd1-80da-4253-b87a-c8707aa3e0b0/68017b66-d25d-4af8-bffb-a371ea1e6e65"
-					(reference "#PWR0149")
-					(unit 1)
-				)
-				(path "/a02e5dd1-80da-4253-b87a-c8707aa3e0b0/d75b9ede-8115-4a1a-ba5c-5202cedca149"
-					(reference "#PWR0142")
+					(reference "#PWR0160")
+					(unit 1)
+				)
+				(path "/a02e5dd1-80da-4253-b87a-c8707aa3e0b0/d75b9ede-8115-4a1a-ba5c-5202cedca149"
+					(reference "#PWR0155")
 					(unit 1)
 				)
@@
 					(unit 1)
 				)
+			)
+		)
+	)
+	(symbol
+		(lib_id "fab_CON:WE_620303124022")
+		(at 204.47 85.09 0)
+		(mirror y)
+		(unit 1)
+		(exclude_from_sim no)
+		(in_bom yes)
+		(on_board yes)
+		(dnp no)
+		(property "Reference" "J15"
+			(at 205.74 86.3601 0)
+			(effects
+				(font
+					(size 1.27 1.27)
+				)
+				(justify right)
+			)
+		)
+		(property "Value" "Conn_01x03_Pin"
+			(at 205.74 83.8201 0)
+			(effects
+				(font
+					(size 1.27 1.27)
+				)
+				(justify right)
+			)
+		)
+		(property "Footprint" "fab_CON:WE_620303124022"
+			(at 204.47 85.09 0)
+			(effects
+				(font
+					(size 1.27 1.27)
+				)
+				(hide yes)
+			)
+		)
+		(property "Datasheet" "https://jlcpcb.com/api/file/downloadByFileSystemAccessId/8589834857439666176"
+			(at 204.47 85.09 0)
+			(effects
+				(font
+					(size 1.27 1.27)
+				)
+				(hide yes)
+			)
+		)
+		(property "Description" "-25℃~+85℃ 1 12mm 1x4P 250V 2A 2mm 3 3P 6.2mm 7.5mm Auxiliary Solder Pin Beige Brass LCP PH Surface Mount,Vertical SMD,P=2mm Wire To Board Connector ROHS"
+			(at 204.47 85.09 0)
+			(effects
+				(font
+					(size 1.27 1.27)
+				)
+				(hide yes)
+			)
+		)
+		(property "LCSC" "C3029432"
+			(at 204.47 85.09 0)
+			(effects
+				(font
+					(size 1.27 1.27)
+				)
+				(hide yes)
+			)
+		)
+		(property "WE" "620303124022"
+			(at 204.47 85.09 0)
+			(effects
+				(font
+					(size 1.27 1.27)
+				)
+				(hide yes)
+			)
+		)
+		(property "Manufacturer" "XUNPU"
+			(at 204.47 85.09 0)
+			(effects
+				(font
+					(size 1.27 1.27)
+				)
+				(hide yes)
+			)
+		)
+		(property "Type" "WAFER-PH2.0-3PLB"
+			(at 204.47 85.09 0)
+			(effects
+				(font
+					(size 1.27 1.27)
+				)
+				(hide yes)
+			)
+		)
+		(pin "1"
+		)
+		(pin "2"
+		)
+		(pin "3"
+		)
+		(instances
+			(project "pnp32_mainboard"
+				(path "/a02e5dd1-80da-4253-b87a-c8707aa3e0b0/68017b66-d25d-4af8-bffb-a371ea1e6e65"
+					(reference "J16")
+					(unit 1)
+				)
+				(path "/a02e5dd1-80da-4253-b87a-c8707aa3e0b0/d75b9ede-8115-4a1a-ba5c-5202cedca149"
+					(reference "J15")
+					(unit 1)
+				)
